File: Furnace_Controller_V1/5v_power_converter.kicad_sch (KiCad schematic)
At the start: 11 parts, among them U2 LM2596S-5, U6 TVS3300DRV

Commit message: V2 dev
Parts:
- removed C1: 220u, Capacitor_THT:CP_Radial_D12.5mm_P5.00mm, symbol Device:C_Polarized
- removed C3: 47u, Capacitor_THT:CP_Radial_D8.0mm_P2.50mm, symbol Device:C_Polarized
- removed D1, D16: 1N5822, Diode_THT:D_DO-201AD_P15.24mm_Horizontal, symbol Diode:1N5822
- removed F2: 3588, MiniAutoFuse:3588, symbol Custom_Symbols:3588
- removed L1: 33u, Coil:SRR1260-150M, symbol Device:L
- removed TP14: 5V_TP, TestPoint:TestPoint_Pad_D1.5mm, symbol Connector:TestPoint
- removed TP26: 24V_TP, TestPoint:TestPoint_Pad_D1.5mm, symbol Connector:TestPoint
- removed U2: LM2596S-5, Package_TO_SOT_SMD:TO-263-5_TabPin3, symbol Regulator_Switching:LM2596S-5
- removed U6: TVS3300DRV, Package_SON:WSON-6-1EP_2x2mm_P0.65mm_EP1x1.6mm, symbol Power_Protection:TVS3300DRV
- added C1, C3: 1u, Capacitor_SMD:C_0805_2012Metric, symbol Device:C
- added C11: 220u, Capacitor_THT:CP_Radial_D12.5mm_P5.00mm, symbol Device:C_Polarized
- added C12: 47u, Capacitor_THT:CP_Radial_D8.0mm_P2.50mm, symbol Device:C_Polarized
- added D19: ss210, Diode_SMD:D_SMA, symbol Diode:SS12
- added L2: 68u, Inductor_SMD:L_10.4x10.4_H4.8, symbol Device:L
- added TP10: 3V3_TP, TestPoint:TestPoint_Pad_D1.0mm, symbol Connector:TestPoint
- added TP19: GND_TP, TestPoint:TestPoint_Pad_D1.0mm, symbol Connector:TestPoint
- added U6: XC6206PxxxMR, Package_TO_SOT_SMD:SOT-23-3, symbol Regulator_Linear:XC6206PxxxMR
- added U7: XL1509-5.0, Package_SO:SOIC-8_3.9x4.9mm_P1.27mm, symbol Regulator_Switching:XL1509-5.0
- TP2: value PGND_TP -> 5V_TP; footprint TestPoint:TestPoint_Pad_D1.5mm -> TestPoint:TestPoint_Pad_D1.0mm
Connections:
- net +5V: now also TP2.1, C1.1, C11.1, L2.2, U6.3 (VI), U7.3 (FB)
- net Logic_GND: now also C11.2, C12.2, D19.2 (A), TP19.1, U7.4 (~{EN}), U7.5 (GND), U7.6 (GND), U7.7 (GND), U7.8 (GND); no longer TP2.1
- net Power In: now also C12.1, U7.1 (VIN)
- new net: C1.2, C3.2, U6.1 (GND)
- new net: D19.1 (K), L2.1, U7.2 (OUT)
- new net +3V3: C3.1, TP10.1, U6.2 (VO)
