File: Furnace_Controller_V1/Furnace_Controller.kicad_pcb (KiCad board)
At the start: 2 copper layers, 149 x 141 mm, 99 parts, among them J1 Power In Treminal, J3 Relay Terminal, J4 HMD Terminal, J5 RS-485 Terminal, Q1 IRLZ44N, Q2 IRLZ44N, Q3 IRLZ44N, Q4 IRLZ44N, Q5 2n2222, U2 LM2596S-5, U3 THVD2450DR, U4 TXU0101DBVR, U5 TXU0101DBVR, U6 TVS3300DRV

Commit message: V2 dev
Parts:
- removed BZ1: Buzzer, Buzzer_Beeper:Buzzer_15x7.5RM7.6
- removed C4: 10u, Capacitor_THT:CP_Radial_D5.0mm_P2.00mm
- removed F2: 3588, MiniAutoFuse:3588
- removed L1: 33u, Coil:SRR1260-150M
- removed TP11, TP5, TP7, TP8, TP9: LGND_TP, TestPoint:TestPoint_Pad_D1.5mm
- removed TP14, TP20: 5V_TP, TestPoint:TestPoint_Pad_D1.5mm
- removed TP21: 3V3_TP, TestPoint:TestPoint_Pad_D1.5mm
- added C11: 220u, Capacitor_THT:CP_Radial_D12.5mm_P5.00mm, F.Cu at (28.0, 24.1)
- added C12: 47u, Capacitor_THT:CP_Radial_D8.0mm_P2.50mm, F.Cu at (22.0, 43.6)
- added C13: 100n, Capacitor_SMD:C_0603_1608Metric, F.Cu at (82.0, 26.2)
- added D20: SM4007, Diode_SMD:D_SOD-123, F.Cu at (88.8, 62.4)
- added D21: SM4007, Diode_SMD:D_SOD-123, F.Cu at (75.8, 60.6)
- added D22: SM4007, Diode_SMD:D_SOD-123, F.Cu at (88.8, 72.0)
- added J11: Conn_01x04_Socket, Connector_PinHeader_2.54mm:PinHeader_1x04_P2.54mm_Vertical, F.Cu at (18.2, 57.0)
- added J2: Relay Terminal, Connector_Phoenix_MC:PhoenixContact_MC_1,5_2-G-3.5_1x02_P3.50mm_Horizontal, F.Cu at (96.5, 54.6)
- added J6: Relay Terminal, Connector_Phoenix_MC:PhoenixContact_MC_1,5_2-G-3.5_1x02_P3.50mm_Horizontal, F.Cu at (96.5, 73.8)
- added J7: Relay Terminal, Connector_Phoenix_MC:PhoenixContact_MC_1,5_2-G-3.5_1x02_P3.50mm_Horizontal, F.Cu at (74.1, 68.5)
- added J8: Relay Terminal, Connector_Phoenix_MC:PhoenixContact_MC_1,5_2-G-3.5_1x02_P3.50mm_Horizontal, F.Cu at (64.5, 68.5)
- added J9: Relay Terminal, Connector_Phoenix_MC:PhoenixContact_MC_1,5_2-G-3.5_1x02_P3.50mm_Horizontal, F.Cu at (54.9, 68.5)
- added JP1: Jumper_2_Open, TestPoint:TestPoint_2Pads_Pitch2.54mm_Drill0.8mm, F.Cu at (29.6, 49.4)
- added L2: 68u, Inductor_SMD:L_10.4x10.4_H4.8, F.Cu at (32.4, 41.4)
- added Q6: HL3402, Package_TO_SOT_SMD:TSOT-23, F.Cu at (52.4, 63.8)
- added R2: 15, Resistor_SMD:R_0603_1608Metric, F.Cu at (78.8, 38.0)
- added R26: 10k, Resistor_SMD:R_0603_1608Metric, F.Cu at (79.4, 41.6)
- added R27: 68, Resistor_SMD:R_0603_1608Metric, F.Cu at (75.4, 44.8)
- added R28: 68, Resistor_SMD:R_0603_1608Metric, F.Cu at (73.4, 44.8)
- added R29: 68, Resistor_SMD:R_0603_1608Metric, F.Cu at (71.4, 44.8)
- added R30: 10k, Resistor_SMD:R_0603_1608Metric, F.Cu at (77.6, 41.6)
- added R31: 10k, Resistor_SMD:R_0603_1608Metric, F.Cu at (71.0, 23.2)
- added R32: 10k, Resistor_SMD:R_0603_1608Metric, F.Cu at (72.8, 23.2)
- added R33: 10k, Resistor_SMD:R_0603_1608Metric, F.Cu at (80.2, 26.2)
- added R34: 10k, Resistor_SMD:R_0603_1608Metric, F.Cu at (53.6, 44.4)
- added R35: 10k, Resistor_SMD:R_0603_1608Metric, F.Cu at (62.6, 44.5)
- added R36: 10k, Resistor_SMD:R_0603_1608Metric, F.Cu at (60.8, 44.4)
- added R37: 10k, Resistor_SMD:R_0603_1608Metric, F.Cu at (51.8, 44.4)
- added R38: 10k, Resistor_SMD:R_0603_1608Metric, F.Cu at (59.0, 44.4)
- added R39: 10k, Resistor_SMD:R_0603_1608Metric, F.Cu at (55.4, 44.4)
- added R40: 10k, Resistor_SMD:R_0603_1608Metric, F.Cu at (57.2, 44.4)
- added SW1: SW_Push, Button_Switch_THT:SW_PUSH_6mm_H4.3mm, F.Cu at (17.8, 68.0)
- added TP10: 3V3_TP, TestPoint:TestPoint_Pad_D1.0mm, F.Cu at (40.2, 25.0)
- added TP28: HR_TP, TestPoint:TestPoint_Pad_D1.0mm, F.Cu at (46.4, 67.0)
- added U7: XL1509-5.0, Package_SO:SOIC-8_3.9x4.9mm_P1.27mm, F.Cu at (29.0, 32.0)
- C1: value 220u -> 1u; footprint Capacitor_THT:CP_Radial_D12.5mm_P5.00mm -> Capacitor_SMD:C_0805_2012Metric
- C2, C5, C6, C7, C8, C9: footprint Capacitor_SMD:C_0805_2012Metric_Pad1.18x1.45mm_HandSolder -> Capacitor_SMD:C_0603_1608Metric
- C3: value 47u -> 1u; footprint Capacitor_THT:CP_Radial_D8.0mm_P2.50mm -> Capacitor_SMD:C_0805_2012Metric
- D1: value 1N5822 -> LED; footprint Diode_THT:D_DO-201AD_P15.24mm_Horizontal -> LED_SMD:LED_0603_1608Metric
- D10, D12, D13, D14, D15, D3, D5, D6, D8: footprint LED_SMD:LED_0805_2012Metric -> LED_SMD:LED_0603_1608Metric
- D11: value LED -> SM4007; footprint LED_SMD:LED_0805_2012Metric -> Diode_SMD:D_SOD-123
- D16: value 1N5822 -> SM4007; footprint Diode_THT:D_DO-201AD_P15.24mm_Horizontal -> Diode_SMD:D_SOD-123
- D19: value 1N4148 -> ss210; footprint Diode_THT:D_DO-35_SOD27_P7.62mm_Horizontal -> Diode_SMD:D_SMA
- D2, D4, D7: value 1N4148 -> LED; footprint Diode_THT:D_DO-35_SOD27_P7.62mm_Horizontal -> LED_SMD:LED_0603_1608Metric
- D9: value 1N4148 -> SM4007; footprint Diode_THT:D_DO-35_SOD27_P7.62mm_Horizontal -> Diode_SMD:D_SOD-123
- J1: footprint TerminalBlock:TerminalBlock_MaiXu_MX126-5.0-02P_1x02_P5.00mm -> Connector_Phoenix_MC:PhoenixContact_MC_1,5_2-G-3.5_1x02_P3.50mm_Horizontal
- J3: footprint TerminalBlock:TerminalBlock_MaiXu_MX126-5.0-09P_1x09_P5.00mm -> Connector_Phoenix_MC:PhoenixContact_MC_1,5_2-G-3.5_1x02_P3.50mm_Horizontal
- J4, J5: footprint TerminalBlock:TerminalBlock_MaiXu_MX126-5.0-04P_1x04_P5.00mm -> Connector_Phoenix_MC:PhoenixContact_MC_1,5_4-G-3.5_1x04_P3.50mm_Horizontal
- Q1, Q2, Q3, Q4: value IRLZ44N -> HL3402; footprint Package_TO_SOT_THT:TO-220-3_Vertical -> Package_TO_SOT_SMD:TSOT-23
- Q5: value 2n2222 -> HL3402; footprint Package_TO_SOT_THT:TO-92_Inline -> Package_TO_SOT_SMD:TSOT-23
- R1: value 10k -> 68; footprint Resistor_SMD:R_0805_2012Metric_Pad1.20x1.40mm_HandSolder -> Resistor_SMD:R_0603_1608Metric
- R10, R11, R12, R13, R14, R15, R20, R21, R22, R23, R24, R4, R5, R6, R7, R8, R9: footprint Resistor_SMD:R_0805_2012Metric_Pad1.20x1.40mm_HandSolder -> Resistor_SMD:R_0603_1608Metric
- R16: value 15 -> 47k; footprint Resistor_SMD:R_0805_2012Metric_Pad1.20x1.40mm_HandSolder -> Resistor_SMD:R_0603_1608Metric
- R17: value 15 -> 68; footprint Resistor_SMD:R_0805_2012Metric_Pad1.20x1.40mm_HandSolder -> Resistor_SMD:R_0603_1608Metric
- R18: value 68 -> 100; footprint Resistor_SMD:R_0805_2012Metric_Pad1.20x1.40mm_HandSolder -> Resistor_SMD:R_0603_1608Metric
- R19: value 68 -> 47k; footprint Resistor_SMD:R_0805_2012Metric_Pad1.20x1.40mm_HandSolder -> Resistor_SMD:R_0603_1608Metric
- R25: value 1k -> 15; footprint Resistor_SMD:R_0805_2012Metric_Pad1.20x1.40mm_HandSolder -> Resistor_SMD:R_0603_1608Metric
- R3: value 10k -> 100; footprint Resistor_SMD:R_0805_2012Metric_Pad1.20x1.40mm_HandSolder -> Resistor_SMD:R_0603_1608Metric
- TP1, TP12, TP13, TP15, TP16, TP18, TP22, TP23, TP24, TP25, TP3, TP4, TP6: footprint TestPoint:TestPoint_Pad_D1.5mm -> TestPoint:TestPoint_Pad_D1.0mm
- TP19: value 3V3_TP -> GND_TP; footprint TestPoint:TestPoint_Pad_D1.5mm -> TestPoint:TestPoint_Pad_D1.0mm
- TP2: value PGND_TP -> 5V_TP; footprint TestPoint:TestPoint_Pad_D1.5mm -> TestPoint:TestPoint_Pad_D1.0mm
- TP26: value 24V_TP -> HR_TP; footprint TestPoint:TestPoint_Pad_D1.5mm -> TestPoint:TestPoint_Pad_D1.0mm
- U1: value ~ -> ESP32-WROOM-32E-N8; footprint Custom_Footprints:ESP32_DevKitc_V4 -> RF_Module:ESP32-WROOM-32
- U2: value LM2596S-5 -> SP3485EN; footprint Package_TO_SOT_SMD:TO-263-5_TabPin3 -> Package_SO:SOIC-8_3.9x4.9mm_P1.27mm
- U3: value THVD2450DR -> W25Q128JVS; footprint THVD:SOIC127P600X175-8N -> Package_SO:SOIC-8_5.3x5.3mm_P1.27mm
- U6: value TVS3300DRV -> XC6206PxxxMR; footprint Package_SON:WSON-6-1EP_2x2mm_P0.65mm_EP1x1.6mm -> Package_TO_SOT_SMD:SOT-23-3
- moved H3 287.5 mm to (331.8, 64.3)
- moved H1 274.0 mm to (331.8, 40.0)
- moved H4 163.5 mm to (331.8, 76.5)
- moved TP19 156.2 mm to (37.4, 27.4), turned to 90 degrees
- moved H2 145.1 mm to (331.8, 52.2)
- moved J5 144.4 mm to (96.5, 28.4)
- moved TP13 144.0 mm to (84.8, 25.6)
- moved D17 143.8 mm to (87.8, 26.8)
- moved D18 142.7 mm to (87.8, 19.2)
- moved R17 142.3 mm to (44.8, 64.4), turned to 90 degrees
- moved R24 142.3 mm to (84.8, 23.0)
- moved TP12 138.2 mm to (84.8, 20.2)
- moved U3 135.2 mm to (74.6, 27.8)
- moved C7 134.8 mm to (53.4, 55.8), turned to -90 degrees
- moved D15 133.2 mm to (55.8, 57.8), turned to 180 degrees
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Connections:
- C1 pad 2: Logic_GND -> Net-(U6-GND)
- C10 pad 1: +5V -> +3V3
- C2 pad 1: +3.3V -> +3V3
- C3 pad 1: +24V -> +3V3
- C3 pad 2: Logic_GND -> Net-(U6-GND)
- C5 pad 1: +3.3V -> +3V3
- C8 pad 1: +3.3V -> +3V3
- C9 pad 1: +5V -> +3V3
- D1 pad 2: Logic_GND -> /Aux3_Relay_Pin
- D10 pad 2: /UART2_TX -> /Aux4_Relay_Pin
- D11 pad 1: Net-(D11-K) -> +24V
- D11 pad 2: /UART2_RX -> /Relay Driver5/Relay-
- D16 pad 1: Net-(D16-K) -> +24V
- D16 pad 2: /5V Power Converter/Power In -> /Relay Driver/Relay-
- D19 pad 1: +5V -> Net-(D19-K)
- D19 pad 2: Net-(BZ1--) -> Logic_GND
- D2 pad 1: +24V -> Net-(D2-K)
- D2 pad 2: /Relay Driver/Relay- -> /UART2_RX
- D4 pad 1: +24V -> Net-(D4-K)
- D4 pad 2: /Relay Driver2/Relay- -> /RS_485_DIR
- D7 pad 1: +24V -> Net-(D7-K)
- D7 pad 2: /Relay Driver3/Relay- -> /UART2_TX
- D9 pad 2: /Relay Driver1/Relay- -> /Relay Driver4/Relay-
- J1 pad 2: /5V Power Converter/Power In -> +24V
- J3 pad 1: Relay_GND -> /Relay Driver1/Relay-
- J3 pad 2: /Relay Driver3/Relay- -> +24V
- Q1 pad 3: Relay_GND -> Logic_GND
- Q2 pad 3: Relay_GND -> Logic_GND
- Q3 pad 3: Relay_GND -> Logic_GND
- Q4 pad 3: Relay_GND -> Logic_GND
- Q5 pad 1: Net-(BZ1--) -> Net-(Q5-G)
- Q5 pad 2: Net-(Q5-B) -> /Relay Driver4/Relay-
- R1 pad 1: +3.3V -> Net-(D1-K)
- R1 pad 2: /UART2_RX -> Logic_GND
- R16 pad 1: /RS-485 Transeiver/RS-485_B -> Net-(Q5-G)
- R16 pad 2: Net-(U3-B) -> Logic_GND
- R17 pad 1: /RS-485 Transeiver/RS-485_A -> Net-(D10-K)
- R17 pad 2: Net-(U3-A) -> Logic_GND
- R18 pad 1: Net-(D10-K) -> /Aux4_Relay_Pin
- R18 pad 2: Logic_GND -> Net-(Q6-G)
- R19 pad 1: Net-(D11-K) -> Net-(Q6-G)
- R25 pad 1: Net-(U1-GPIO23) -> /RS-485 Transeiver/RS-485_B
- R25 pad 2: Net-(Q5-B) -> Net-(U2-B)
- R3 pad 1: /RS_485_DIR -> /Aux3_Relay_Pin
- R3 pad 2: Logic_GND -> Net-(Q5-G)
- TP19 pad 1: +3.3V -> Logic_GND
- TP2 pad 1: Logic_GND -> +5V
- TP26 pad 1: +24V -> /Aux3_Relay_Pin
- U1 pad 1: +3.3V -> Logic_GND
- U1 pad 10: /UART2_RX -> /UART1_TX
- U1 pad 11: /UART2_TX -> /UART1_RX
- U1 pad 12: unconnected-(U1-GPIO14-Pad12) -> /Heater_Relay_Pin
- U1 pad 13: unconnected-(U1-GPIO12-Pad13) -> /Fan_Relay_Pin
- U1 pad 14: Logic_GND -> Net-(U1-IO12)
- U1 pad 15: unconnected-(U1-GPIO13-Pad15) -> Logic_GND
- U1 pad 16: unconnected-(U1-GPIO9-Pad16) -> /Aux_Relay_Pin
- U1 pad 17: unconnected-(U1-GPIO10-Pad17) -> Net-(U1-SHD/SD2)
- U1 pad 18: unconnected-(U1-GPIO11-Pad18) -> Net-(U1-SWP/SD3)
- U1 pad 19: +5V -> unconnected-(U1-SCS/CMD-Pad19)
- U1 pad 2: unconnected-(U1-EN-Pad2) -> +3V3
- U1 pad 23: unconnected-(U1-GPIO15-Pad23) -> Net-(U1-IO15)
- U1 pad 24: unconnected-(U1-GPIO2-Pad24) -> Net-(U1-IO2)
- U1 pad 25: unconnected-(U1-GPIO0-Pad25) -> Net-(U1-IO0)
- U1 pad 26: unconnected-(U1-GPIO4-Pad26) -> /UART2_TX
- U1 pad 27: /UART1_RX -> /RS_485_DIR
- U1 pad 28: /UART1_TX -> /UART2_RX
- U1 pad 29: unconnected-(U1-GPIO5-Pad29) -> /BUZZER
- U1 pad 3: unconnected-(U1-GPIO36-Pad3) -> Net-(U1-EN)
- U1 pad 30: /Aux2_Relay_Pin -> /SPI_MOSI
- U1 pad 31: /Aux_Relay_Pin -> /SPI_CLK
- U1 pad 32: Logic_GND -> unconnected-(U1-NC-Pad32)
- U1 pad 33: /Fan_Relay_Pin -> /SPI_MISO
- U1 pad 34: unconnected-(U1-GPIO3/U0RXD-Pad34) -> /UART0_RX
- U1 pad 35: unconnected-(U1-GPIO1/U0TXD-Pad35) -> /UART0_TX
- U1 pad 36: /Heater_Relay_Pin -> /Aux4_Relay_Pin
- U1 pad 37: Net-(U1-GPIO23) -> /FLASH_CS
- U1 pad 8: unconnected-(U1-GPIO33-Pad8) -> /Aux3_Relay_Pin
- U1 pad 9: /RS_485_DIR -> /Aux2_Relay_Pin
- U2 pad 1: +24V -> /UART2_RX
- U2 pad 2: Net-(D1-K) -> /RS_485_DIR
- U2 pad 3: Logic_GND -> /RS_485_DIR
- U2 pad 4: +5V -> /UART2_TX
- U3 pad 1: /UART2_RX -> /FLASH_CS
- U3 pad 2: /RS_485_DIR -> /SPI_MISO
- U3 pad 3: /RS_485_DIR -> Net-(U3-~{WP}/IO_{2})
- U3 pad 4: /UART2_TX -> Logic_GND
- U3 pad 5: Logic_GND -> /SPI_MOSI
- U3 pad 6: Net-(U3-A) -> /SPI_CLK
- U3 pad 7: Net-(U3-B) -> Net-(U3-~{HOLD}/~{RESET}/IO_{3})
- U3 pad 8: +3.3V -> +3V3
- U4 pad 5: +3.3V -> +3V3
- U4 pad 6: +3.3V -> +3V3
- U5 pad 1: +3.3V -> +3V3
- U6 pad 1: Logic_GND -> Net-(U6-GND)
- U6 pad 2: Logic_GND -> +3V3
- U6 pad 3: Logic_GND -> +5V
Routing:
- net +5V: track 295.2 -> 64.4 mm, vias 1 -> 4
- net +3.3V: track 149.8 -> 0.00 mm, vias 3 -> 0
- net +24V: track 294.7 -> 175.7 mm
- net +3V3: track 0.00 -> 117.4 mm, vias 0 -> 6
- net /UART2_TX: track 93.4 -> 9.13 mm
- net /RS_485_DIR: track 97.2 -> 24.2 mm
- net /UART2_RX: track 89.6 -> 18.9 mm
- net Net-(U1-GPIO23): track 65.3 -> 0.00 mm, vias 1 -> 0
- net /Nextion Level Shifter/HMD_RX: track 17.0 -> 81.6 mm
- net Relay_GND: track 60.1 -> 0.00 mm
- net /Nextion Level Shifter/HMD_TX: track 17.0 -> 71.7 mm
- net Net-(D19-K): track 0.00 -> 26.2 mm
- net /Aux2_Relay_Pin: track 34.7 -> 8.62 mm, vias 0 -> 1
- net /UART1_RX: track 60.4 -> 34.8 mm
- net /Aux_Relay_Pin: track 25.1 -> 0.00 mm
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- added copper zone on In2.Cu, net +5V
- added copper zone on In1.Cu, net Logic_GND
Other:
- board size 149 x 141 mm -> 90 x 62.2 mm
- copper layers 2 -> 4
- board text added: "24V"
- board text added: "24V+"
- board text added: "3V3"
- board text added: "5V"
- board text added: "A"
- board text added: "AUX1"
- board text added: "AUX2"
- board text added: "AUX3"
- board text added: "AUX4"
- board text added: "B"
- board text added: "BOOT"
- board text added: "FAN"
- board text added: "GND"
- board text added: "HEATER"
- board text added: "HMI_RX_H"
- board text added: "HMI_RX_L"
- board text added: "HMI_TX_H"
- board text added: "HMI_TX_L"
- board text added: "PIN"
- board text added: "POWER_EN"
- board text added: "RLY-"
- board text added: "RS_DIR"
- board text added: "RS_RX"
- board text added: "RS_TX"
- board text added: "RX"
- board text added: "TX"
- board text added: "UART0_RX"
- board text added: "UART0_TX"
- board text removed: "V1.0P"
- board text removed: "VT KA SK"
- board text removed: "telamorph.com"
- board text removed: "мойтапечка.com"
