File: Furnace_Controller_V1/Furnace_Controller.kicad_pcb (KiCad board)
At the start: 4 copper layers, 90 x 62.2 mm, 122 parts, among them J1 Power In Treminal, J11 Conn_01x04_Socket, J2 Relay Terminal, J3 Relay Terminal, J4 HMD Terminal, J5 RS-485 Terminal, J6 Relay Terminal, J7 Relay Terminal, J8 Relay Terminal, J9 Relay Terminal, Q1 HL3402, Q2 HL3402, Q3 HL3402, Q4 HL3402, Q5 HL3402, Q6 HL3402, SW1 SW_Push, U1 ESP32-WROOM-32E-N8, U2 SP3485EN, U3 W25Q128JVS, U4 TXU0101DBVR, U5 TXU0101DBVR, U6 XC6206PxxxMR, U7 XL1509-5.0

Commit message: Organize PCB revisions and correct TI footprints
Parts:
- removed C11: 220u, Capacitor_THT:CP_Radial_D12.5mm_P5.00mm
- removed C12: 47u, Capacitor_THT:CP_Radial_D8.0mm_P2.50mm
- removed C13: 100n, Capacitor_SMD:C_0603_1608Metric
- removed D20, D21, D22: SM4007, Diode_SMD:D_SOD-123
- removed J11: Conn_01x04_Socket, Connector_PinHeader_2.54mm:PinHeader_1x04_P2.54mm_Vertical
- removed J2, J6, J7, J8, J9: Relay Terminal, Connector_Phoenix_MC:PhoenixContact_MC_1,5_2-G-3.5_1x02_P3.50mm_Horizontal
- removed JP1: Jumper_2_Open, TestPoint:TestPoint_2Pads_Pitch2.54mm_Drill0.8mm
- removed L2: 68u, Inductor_SMD:L_10.4x10.4_H4.8
- removed Q6: HL3402, Package_TO_SOT_SMD:TSOT-23
- removed R2: 15, Resistor_SMD:R_0603_1608Metric
- removed R26, R30, R31, R32, R33, R34, R35, R36, R37, R38, R39, R40: 10k, Resistor_SMD:R_0603_1608Metric
- removed R27, R28, R29: 68, Resistor_SMD:R_0603_1608Metric
- removed SW1: SW_Push, Button_Switch_THT:SW_PUSH_6mm_H4.3mm
- removed TP10: 3V3_TP, TestPoint:TestPoint_Pad_D1.0mm
- removed TP28: HR_TP, TestPoint:TestPoint_Pad_D1.0mm
- removed U7: XL1509-5.0, Package_SO:SOIC-8_3.9x4.9mm_P1.27mm
- added BZ1: Buzzer, Buzzer_Beeper:Buzzer_15x7.5RM7.6, F.Cu at (68.5, 83.8)
- added C4: 10u, Capacitor_THT:CP_Radial_D5.0mm_P2.00mm, F.Cu at (133.0, 118.3)
- added F2: 3588, MiniAutoFuse:3588, F.Cu at (69.5, 65.1)
- added L1: 33u, Coil:SRR1260-150M, F.Cu at (39.5, 48.6)
- added TP11: LGND_TP, TestPoint:TestPoint_Pad_D1.5mm, F.Cu at (133.0, 134.8)
- added TP14: 5V_TP, TestPoint:TestPoint_Pad_D1.5mm, F.Cu at (42.0, 59.6)
- added TP20: 5V_TP, TestPoint:TestPoint_Pad_D1.5mm, F.Cu at (144.0, 87.3)
- added TP21: 3V3_TP, TestPoint:TestPoint_Pad_D1.5mm, F.Cu at (141.0, 108.8)
- added TP5: LGND_TP, TestPoint:TestPoint_Pad_D1.5mm, F.Cu at (129.5, 67.3)
- added TP7: LGND_TP, TestPoint:TestPoint_Pad_D1.5mm, F.Cu at (129.5, 42.3)
- added TP8: LGND_TP, TestPoint:TestPoint_Pad_D1.5mm, F.Cu at (129.5, 79.8)
- added TP9: LGND_TP, TestPoint:TestPoint_Pad_D1.5mm, F.Cu at (129.5, 54.8)
- C1: value 1u -> 220u; footprint Capacitor_SMD:C_0805_2012Metric -> Capacitor_THT:CP_Radial_D12.5mm_P5.00mm
- C2, C5, C6, C7, C8, C9: footprint Capacitor_SMD:C_0603_1608Metric -> Capacitor_SMD:C_0805_2012Metric_Pad1.18x1.45mm_HandSolder
- C3: value 1u -> 47u; footprint Capacitor_SMD:C_0805_2012Metric -> Capacitor_THT:CP_Radial_D8.0mm_P2.50mm
- D1: value LED -> 1N5822; footprint LED_SMD:LED_0603_1608Metric -> Diode_THT:D_DO-201AD_P15.24mm_Horizontal
- D10, D12, D13, D14, D15, D3, D5, D6, D8: footprint LED_SMD:LED_0603_1608Metric -> LED_SMD:LED_0805_2012Metric
- D11: value SM4007 -> LED; footprint Diode_SMD:D_SOD-123 -> LED_SMD:LED_0805_2012Metric
- D16: value SM4007 -> 1N5822; footprint Diode_SMD:D_SOD-123 -> Diode_THT:D_DO-201AD_P15.24mm_Horizontal
- D19: value ss210 -> 1N4148; footprint Diode_SMD:D_SMA -> Diode_THT:D_DO-35_SOD27_P7.62mm_Horizontal
- D2, D4, D7: value LED -> 1N4148; footprint LED_SMD:LED_0603_1608Metric -> Diode_THT:D_DO-35_SOD27_P7.62mm_Horizontal
- D9: value SM4007 -> 1N4148; footprint Diode_SMD:D_SOD-123 -> Diode_THT:D_DO-35_SOD27_P7.62mm_Horizontal
- J1: footprint Connector_Phoenix_MC:PhoenixContact_MC_1,5_2-G-3.5_1x02_P3.50mm_Horizontal -> TerminalBlock:TerminalBlock_MaiXu_MX126-5.0-02P_1x02_P5.00mm
- J3: footprint Connector_Phoenix_MC:PhoenixContact_MC_1,5_2-G-3.5_1x02_P3.50mm_Horizontal -> TerminalBlock:TerminalBlock_MaiXu_MX126-5.0-09P_1x09_P5.00mm
- J4, J5: footprint Connector_Phoenix_MC:PhoenixContact_MC_1,5_4-G-3.5_1x04_P3.50mm_Horizontal -> TerminalBlock:TerminalBlock_MaiXu_MX126-5.0-04P_1x04_P5.00mm
- Q1, Q2, Q3, Q4: value HL3402 -> IRLZ44N; footprint Package_TO_SOT_SMD:TSOT-23 -> Package_TO_SOT_THT:TO-220-3_Vertical
- Q5: value HL3402 -> 2n2222; footprint Package_TO_SOT_SMD:TSOT-23 -> Package_TO_SOT_THT:TO-92_Inline
- R1: value 68 -> 10k; footprint Resistor_SMD:R_0603_1608Metric -> Resistor_SMD:R_0805_2012Metric_Pad1.20x1.40mm_HandSolder
- R10, R11, R12, R13, R14, R15, R20, R21, R22, R23, R24, R4, R5, R6, R7, R8, R9: footprint Resistor_SMD:R_0603_1608Metric -> Resistor_SMD:R_0805_2012Metric_Pad1.20x1.40mm_HandSolder
- R16: value 47k -> 15; footprint Resistor_SMD:R_0603_1608Metric -> Resistor_SMD:R_0805_2012Metric_Pad1.20x1.40mm_HandSolder
- R17: value 68 -> 15; footprint Resistor_SMD:R_0603_1608Metric -> Resistor_SMD:R_0805_2012Metric_Pad1.20x1.40mm_HandSolder
- R18: value 100 -> 68; footprint Resistor_SMD:R_0603_1608Metric -> Resistor_SMD:R_0805_2012Metric_Pad1.20x1.40mm_HandSolder
- R19: value 47k -> 68; footprint Resistor_SMD:R_0603_1608Metric -> Resistor_SMD:R_0805_2012Metric_Pad1.20x1.40mm_HandSolder
- R25: value 15 -> 1k; footprint Resistor_SMD:R_0603_1608Metric -> Resistor_SMD:R_0805_2012Metric_Pad1.20x1.40mm_HandSolder
- R3: value 100 -> 10k; footprint Resistor_SMD:R_0603_1608Metric -> Resistor_SMD:R_0805_2012Metric_Pad1.20x1.40mm_HandSolder
- TP1, TP12, TP13, TP15, TP16, TP18, TP22, TP23, TP24, TP25, TP3, TP4, TP6: footprint TestPoint:TestPoint_Pad_D1.0mm -> TestPoint:TestPoint_Pad_D1.5mm
- TP19: value GND_TP -> 3V3_TP; footprint TestPoint:TestPoint_Pad_D1.0mm -> TestPoint:TestPoint_Pad_D1.5mm
- TP2: value 5V_TP -> PGND_TP; footprint TestPoint:TestPoint_Pad_D1.0mm -> TestPoint:TestPoint_Pad_D1.5mm
- TP26: value HR_TP -> 24V_TP; footprint TestPoint:TestPoint_Pad_D1.0mm -> TestPoint:TestPoint_Pad_D1.5mm
- U1: value ESP32-WROOM-32E-N8 -> ~; footprint RF_Module:ESP32-WROOM-32 -> Custom_Footprints:ESP32_DevKitc_V4
- U2: value SP3485EN -> LM2596S-5; footprint Package_SO:SOIC-8_3.9x4.9mm_P1.27mm -> Package_TO_SOT_SMD:TO-263-5_TabPin3
- U3: value W25Q128JVS -> THVD2450DR; footprint Package_SO:SOIC-8_5.3x5.3mm_P1.27mm -> THVD:SOIC127P600X175-8N
- U6: value XC6206PxxxMR -> TVS3300DRV; footprint Package_TO_SOT_SMD:SOT-23-3 -> Package_SON:WSON-6-1EP_2x2mm_P0.65mm_EP1x1.6mm
- moved H3 317.0 mm to (26.0, 147.8)
- moved H1 306.2 mm to (26.0, 25.3)
- moved H4 190.8 mm to (155.0, 148.3)
- moved H2 177.4 mm to (156.5, 25.3)
- moved TP19 128.5 mm to (133.0, 113.3), turned to 0 degrees
- moved TP13 122.4 mm to (144.0, 132.8)
- moved J5 122.3 mm to (158.5, 133.8)
- moved D17 121.4 mm to (150.5, 130.8)
- moved D18 120.2 mm to (150.5, 121.8)
- moved R24 120.1 mm to (146.0, 126.3)
- moved TP12 115.9 mm to (144.0, 119.8)
- moved U3 113.2 mm to (130.5, 126.3)
- moved R17 112.9 mm to (137.5, 128.8), turned to 180 degrees
- moved C2 105.7 mm to (132.0, 122.3), turned to 180 degrees
- moved C7 104.1 mm to (145.0, 105.3), turned to 0 degrees
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Connections:
- C1 pad 2: Net-(U6-GND) -> Logic_GND
- C10 pad 1: +3V3 -> +5V
- C2 pad 1: +3V3 -> +3.3V
- C3 pad 1: +3V3 -> +24V
- C3 pad 2: Net-(U6-GND) -> Logic_GND
- C5 pad 1: +3V3 -> +3.3V
- C8 pad 1: +3V3 -> +3.3V
- C9 pad 1: +3V3 -> +5V
- D1 pad 2: /Aux3_Relay_Pin -> Logic_GND
- D10 pad 2: /Aux4_Relay_Pin -> /UART2_TX
- D11 pad 1: +24V -> Net-(D11-K)
- D11 pad 2: /Relay Driver5/Relay- -> /UART2_RX
- D16 pad 1: +24V -> Net-(D16-K)
- D16 pad 2: /Relay Driver/Relay- -> /5V Power Converter/Power In
- D19 pad 1: Net-(D19-K) -> +5V
- D19 pad 2: Logic_GND -> Net-(BZ1--)
- D2 pad 1: Net-(D2-K) -> +24V
- D2 pad 2: /UART2_RX -> /Relay Driver/Relay-
- D4 pad 1: Net-(D4-K) -> +24V
- D4 pad 2: /RS_485_DIR -> /Relay Driver2/Relay-
- D7 pad 1: Net-(D7-K) -> +24V
- D7 pad 2: /UART2_TX -> /Relay Driver3/Relay-
- D9 pad 2: /Relay Driver4/Relay- -> /Relay Driver1/Relay-
- J1 pad 2: +24V -> /5V Power Converter/Power In
- J3 pad 1: /Relay Driver1/Relay- -> Relay_GND
- J3 pad 2: +24V -> /Relay Driver3/Relay-
- Q1 pad 3: Logic_GND -> Relay_GND
- Q2 pad 3: Logic_GND -> Relay_GND
- Q3 pad 3: Logic_GND -> Relay_GND
- Q4 pad 3: Logic_GND -> Relay_GND
- Q5 pad 1: Net-(Q5-G) -> Net-(BZ1--)
- Q5 pad 2: /Relay Driver4/Relay- -> Net-(Q5-B)
- R1 pad 1: Net-(D1-K) -> +3.3V
- R1 pad 2: Logic_GND -> /UART2_RX
- R16 pad 1: Net-(Q5-G) -> /RS-485 Transeiver/RS-485_B
- R16 pad 2: Logic_GND -> Net-(U3-B)
- R17 pad 1: Net-(D10-K) -> /RS-485 Transeiver/RS-485_A
- R17 pad 2: Logic_GND -> Net-(U3-A)
- R18 pad 1: /Aux4_Relay_Pin -> Net-(D10-K)
- R18 pad 2: Net-(Q6-G) -> Logic_GND
- R19 pad 1: Net-(Q6-G) -> Net-(D11-K)
- R25 pad 1: /RS-485 Transeiver/RS-485_B -> Net-(U1-GPIO23)
- R25 pad 2: Net-(U2-B) -> Net-(Q5-B)
- R3 pad 1: /Aux3_Relay_Pin -> /RS_485_DIR
- R3 pad 2: Net-(Q5-G) -> Logic_GND
- TP19 pad 1: Logic_GND -> +3.3V
- TP2 pad 1: +5V -> Logic_GND
- TP26 pad 1: /Aux3_Relay_Pin -> +24V
- U1 pad 1: Logic_GND -> +3.3V
- U1 pad 10: /UART1_TX -> /UART2_RX
- U1 pad 11: /UART1_RX -> /UART2_TX
- U1 pad 12: /Heater_Relay_Pin -> unconnected-(U1-GPIO14-Pad12)
- U1 pad 13: /Fan_Relay_Pin -> unconnected-(U1-GPIO12-Pad13)
- U1 pad 14: Net-(U1-IO12) -> Logic_GND
- U1 pad 15: Logic_GND -> unconnected-(U1-GPIO13-Pad15)
- U1 pad 16: /Aux_Relay_Pin -> unconnected-(U1-GPIO9-Pad16)
- U1 pad 17: Net-(U1-SHD/SD2) -> unconnected-(U1-GPIO10-Pad17)
- U1 pad 18: Net-(U1-SWP/SD3) -> unconnected-(U1-GPIO11-Pad18)
- U1 pad 19: unconnected-(U1-SCS/CMD-Pad19) -> +5V
- U1 pad 2: +3V3 -> unconnected-(U1-EN-Pad2)
- U1 pad 23: Net-(U1-IO15) -> unconnected-(U1-GPIO15-Pad23)
- U1 pad 24: Net-(U1-IO2) -> unconnected-(U1-GPIO2-Pad24)
- U1 pad 25: Net-(U1-IO0) -> unconnected-(U1-GPIO0-Pad25)
- U1 pad 26: /UART2_TX -> unconnected-(U1-GPIO4-Pad26)
- U1 pad 27: /RS_485_DIR -> /UART1_RX
- U1 pad 28: /UART2_RX -> /UART1_TX
- U1 pad 29: /BUZZER -> unconnected-(U1-GPIO5-Pad29)
- U1 pad 3: Net-(U1-EN) -> unconnected-(U1-GPIO36-Pad3)
- U1 pad 30: /SPI_MOSI -> /Aux2_Relay_Pin
- U1 pad 31: /SPI_CLK -> /Aux_Relay_Pin
- U1 pad 32: unconnected-(U1-NC-Pad32) -> Logic_GND
- U1 pad 33: /SPI_MISO -> /Fan_Relay_Pin
- U1 pad 34: /UART0_RX -> unconnected-(U1-GPIO3/U0RXD-Pad34)
- U1 pad 35: /UART0_TX -> unconnected-(U1-GPIO1/U0TXD-Pad35)
- U1 pad 36: /Aux4_Relay_Pin -> /Heater_Relay_Pin
- U1 pad 37: /FLASH_CS -> Net-(U1-GPIO23)
- U1 pad 8: /Aux3_Relay_Pin -> unconnected-(U1-GPIO33-Pad8)
- U1 pad 9: /Aux2_Relay_Pin -> /RS_485_DIR
- U2 pad 1: /UART2_RX -> +24V
- U2 pad 2: /RS_485_DIR -> Net-(D1-K)
- U2 pad 3: /RS_485_DIR -> Logic_GND
- U2 pad 4: /UART2_TX -> +5V
- U3 pad 1: /FLASH_CS -> /UART2_RX
- U3 pad 2: /SPI_MISO -> /RS_485_DIR
- U3 pad 3: Net-(U3-~{WP}/IO_{2}) -> /RS_485_DIR
- U3 pad 4: Logic_GND -> /UART2_TX
- U3 pad 5: /SPI_MOSI -> Logic_GND
- U3 pad 6: /SPI_CLK -> Net-(U3-A)
- U3 pad 7: Net-(U3-~{HOLD}/~{RESET}/IO_{3}) -> Net-(U3-B)
- U3 pad 8: +3V3 -> +3.3V
- U4 pad 5: +3V3 -> +3.3V
- U4 pad 6: +3V3 -> +3.3V
- U5 pad 1: +3V3 -> +3.3V
- U6 pad 1: Net-(U6-GND) -> Logic_GND
- U6 pad 2: +3V3 -> Logic_GND
- U6 pad 3: +5V -> Logic_GND
Routing:
- net +5V: track 64.4 -> 295.2 mm, vias 4 -> 1
- net +3.3V: track 0.00 -> 149.8 mm, vias 0 -> 3
- net +24V: track 175.7 -> 294.7 mm
- net +3V3: track 117.4 -> 0.00 mm, vias 6 -> 0
- net /UART2_TX: track 9.13 -> 93.4 mm
- net /RS_485_DIR: track 24.2 -> 97.2 mm
- net /UART2_RX: track 18.9 -> 89.6 mm
- net Net-(U1-GPIO23): track 0.00 -> 65.3 mm, vias 0 -> 1
- net /Nextion Level Shifter/HMD_RX: track 81.6 -> 17.0 mm
- net Relay_GND: track 0.00 -> 60.1 mm
- net /Nextion Level Shifter/HMD_TX: track 71.7 -> 17.0 mm
- net Net-(D19-K): track 26.2 -> 0.00 mm
- net /Aux2_Relay_Pin: track 8.62 -> 34.7 mm, vias 1 -> 0
- net /UART1_RX: track 34.8 -> 60.4 mm
- net /Aux_Relay_Pin: track 0.00 -> 25.1 mm
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- removed copper zone on In2.Cu, net +5V
- removed copper zone on In1.Cu, net Logic_GND
Other:
- board size 90 x 62.2 mm -> 149 x 141 mm
- copper layers 4 -> 2
- board text added: "V1.0P"
- board text added: "VT KA SK"
- board text added: "telamorph.com"
- board text added: "мойтапечка.com"
- board text removed: "24V"
- board text removed: "24V+"
- board text removed: "3V3"
- board text removed: "5V"
- board text removed: "A"
- board text removed: "AUX1"
- board text removed: "AUX2"
- board text removed: "AUX3"
- board text removed: "AUX4"
- board text removed: "B"
- board text removed: "BOOT"
- board text removed: "FAN"
- board text removed: "GND"
- board text removed: "HEATER"
- board text removed: "HMI_RX_H"
- board text removed: "HMI_RX_L"
- board text removed: "HMI_TX_H"
- board text removed: "HMI_TX_L"
- board text removed: "PIN"
- board text removed: "POWER_EN"
- board text removed: "RLY-"
- board text removed: "RS_DIR"
- board text removed: "RS_RX"
- board text removed: "RS_TX"
- board text removed: "RX"
- board text removed: "TX"
- board text removed: "UART0_RX"
- board text removed: "UART0_TX"

Commit message: Normalize 3.3V net names
Connections:
- net +3.3V renamed +3V3
Changed lines of the file:
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@@
 	(net 1 "Net-(BZ1--)")
 	(net 2 "+5V")
-	(net 3 "+3.3V")
+	(net 3 "+3V3")
 	(net 4 "+24V")
 	(net 5 "Logic_GND")
@@
 			(layers "*.Cu" "*.Mask")
 			(remove_unused_layers no)
-			(net 3 "+3.3V")
+			(net 3 "+3V3")
 			(pinfunction "3V3")
 			(pintype "power_out")
@@
 			(size 0.6 1.2)
 			(layers "F.Cu" "F.Mask" "F.Paste")
-			(net 3 "+3.3V")
+			(net 3 "+3V3")
 			(pinfunction "VCCA")
 			(pintype "power_in")
@@
 			(size 1.5 1.5)
 			(layers "F.Cu" "F.Mask")
-			(net 3 "+3.3V")
+			(net 3 "+3V3")
 			(pinfunction "1")
 			(pintype "passive")
@@
 			(layers "F.Cu" "F.Mask" "F.Paste")
 			(roundrect_rratio 0.208333)
-			(net 3 "+3.3V")
+			(net 3 "+3V3")
 			(pintype "passive")
 		)
@@
 			(size 0.6 1.2)
 			(layers "F.Cu" "F.Mask" "F.Paste")
-			(net 3 "+3.3V")
+			(net 3 "+3V3")
 			(pinfunction "OE")
 			(pintype "input")
@@
 			(size 0.6 1.2)
 			(layers "F.Cu" "F.Mask" "F.Paste")
-			(net 3 "+3.3V")
+			(net 3 "+3V3")
 			(pinfunction "VCCB")
 			(pintype "power_in")
@@
 			(size 1.5 1.5)
 			(layers "F.Cu" "F.Mask")
-			(net 3 "+3.3V")
+			(net 3 "+3V3")
 			(pinfunction "1")
 			(pintype "passive")
@@
 			(size 0.65 1.528)
 			(layers "F.Cu" "F.Mask" "F.Paste")
-			(net 3 "+3.3V")
+			(net 3 "+3V3")
 			(pinfunction "VCC")
 			(pintype "power_in")
@@
 			(layers "F.Cu" "F.Mask" "F.Paste")
 			(roundrect_rratio 0.212766)
-			(net 3 "+3.3V")
+			(net 3 "+3V3")
 			(pintype "passive")
 		)
@@
 			(layers "F.Cu" "F.Mask" "F.Paste")
 			(roundrect_rratio 0.212766)
-			(net 3 "+3.3V")
+			(net 3 "+3V3")
 			(pintype "passive")
 		)
@@
 			(layers "F.Cu" "F.Mask" "F.Paste")
 			(roundrect_rratio 0.212766)
-			(net 3 "+3.3V")
+			(net 3 "+3V3")
 			(pintype "passive")
 		)
@@
 			(remove_unused_layers no)
 			(roundrect_rratio 0.15625)
-			(net 3 "+3.3V")
+			(net 3 "+3V3")
 			(pintype "passive")
 		)
