File: Furnace_Controller_V1/Furnace_Controller.kicad_sch (KiCad schematic)
At the start: 18 parts, among them J1 Power In Treminal, J3 Relay Terminal, J4 HMD Terminal, J5 RS-485 Terminal, Q5 2n2222

Commit message: V2 dev
Parts:
- removed BZ1: Buzzer, Buzzer_Beeper:Buzzer_15x7.5RM7.6, symbol Device:Buzzer
- removed D19: 1N4148, Diode_THT:D_DO-35_SOD27_P7.62mm_Horizontal, symbol Diode:1N4148
- removed J3: Relay Terminal, TerminalBlock:TerminalBlock_MaiXu_MX126-5.0-09P_1x09_P5.00mm, symbol Connector:Screw_Terminal_01x09
- removed Q5: 2n2222, Package_TO_SOT_THT:TO-92_Inline, symbol Transistor_BJT:BC337
- removed R25: 1k, Resistor_SMD:R_0805_2012Metric_Pad1.20x1.40mm_HandSolder, symbol Device:R
- removed U1: ~, Custom_Footprints:ESP32_DevKitc_V4, symbol Custom_Symbols:ESP32_DevKitc_V4
- added C13: 100n, Capacitor_SMD:C_0603_1608Metric, symbol Device:C
- added J11: Conn_01x04_Socket, Connector_PinHeader_2.54mm:PinHeader_1x04_P2.54mm_Vertical, symbol Connector:Conn_01x04_Socket
- added J2, J3, J6, J7, J8, J9: Relay Terminal, Connector_Phoenix_MC:PhoenixContact_MC_1,5_2-G-3.5_1x02_P3.50mm_Horizontal, symbol Connector:Screw_Terminal_01x02
- added JP1: Jumper_2_Open, TestPoint:TestPoint_2Pads_Pitch2.54mm_Drill0.8mm, symbol Jumper:Jumper_2_Open
- added R31, R32, R33, R34, R35, R36, R37, R38, R39, R40: 10k, Resistor_SMD:R_0603_1608Metric, symbol Device:R
- added SW1: SW_Push, Button_Switch_THT:SW_PUSH_6mm_H4.3mm, symbol Switch:SW_Push
- added U1: ESP32-WROOM-32E-N8, RF_Module:ESP32-WROOM-32, symbol RF_Module:ESP32-WROOM-32
- added U3: W25Q128JVS, Package_SO:SOIC-8_5.3x5.3mm_P1.27mm, symbol Memory_Flash:W25Q128JVS
- C9: footprint Capacitor_SMD:C_0805_2012Metric_Pad1.18x1.45mm_HandSolder -> Capacitor_SMD:C_0603_1608Metric
- J1: footprint TerminalBlock:TerminalBlock_MaiXu_MX126-5.0-02P_1x02_P5.00mm -> Connector_Phoenix_MC:PhoenixContact_MC_1,5_2-G-3.5_1x02_P3.50mm_Horizontal
- J4, J5: footprint TerminalBlock:TerminalBlock_MaiXu_MX126-5.0-04P_1x04_P5.00mm -> Connector_Phoenix_MC:PhoenixContact_MC_1,5_4-G-3.5_1x04_P3.50mm_Horizontal
- R24: footprint Resistor_SMD:R_0805_2012Metric_Pad1.20x1.40mm_HandSolder -> Resistor_SMD:R_0603_1608Metric
Connections:
- net Power Supply/Power In is gone; now on net +24V: J1.2 (Pin_2)
- net +5V: no longer C10.1, C9.1
- net Aux2_Relay_Pin: now also U1.9 (IO33)
- net Aux_Relay_Pin: now also U1.16 (IO13)
- net Fan_Relay_Pin: now also U1.13 (IO14)
- net Heater_Relay_Pin: now also U1.12 (IO27)
- net Logic_GND: now also C13.2, J11.1 (Pin_1), R38.2, SW1.2, U1.1 (GND), U1.15 (GND), U1.38 (GND), U1.39 (GND), U3.4 (GND)
- net RS_485_DIR: now also U1.27 (IO16)
- net Relay Driver/Relay+: now also J2.2 (Pin_2)
- net Relay Driver/Relay-: now also J2.1 (Pin_1)
- net Relay Driver1/Relay+: now also J3.2 (Pin_2)
- net Relay Driver1/Relay-: now also J3.1 (Pin_1)
- net Relay Driver2/Relay+: now also J6.2 (Pin_2)
- net Relay Driver2/Relay-: now also J6.1 (Pin_1)
- net Relay Driver3/Relay+: now also J7.2 (Pin_2)
- net Relay Driver3/Relay-: now also J7.1 (Pin_1)
- net UART1_RX: now also U1.11 (IO26)
- net UART1_TX: now also U1.10 (IO25)
- net UART2_RX: now also U1.28 (IO17)
- net UART2_TX: now also U1.26 (IO4)
- new net: J11.4 (Pin_4), JP1.2 (B)
- new net: R35.2, SW1.1, U1.25 (IO0)
- new net: R40.2, U1.18 (SWP/SD3)
- new net: R37.2, U1.14 (IO12)
- new net: R39.2, U1.17 (SHD/SD2)
- new net: R38.1, U1.23 (IO15)
- new net: R36.2, U1.24 (IO2)
- new net: R34.2, U1.3 (EN)
- new net: R33.2, U3.7 (~{HOLD}/~{RESET}/IO_{3})
- new net: R32.2, U3.3 (~{WP}/IO_{2})
- new net +3V3: C10.1, C13.1, C9.1, JP1.1 (A), R31.1, R32.1, R33.1, R34.1, R35.1, R36.1, R37.1, R39.1, R40.1, U1.2 (VDD), U3.8 (VCC)
- new net Aux3_Relay_Pin: U1.8 (IO32)
- new net Aux4_Relay_Pin: U1.36 (IO22)
- new net BUZZER: U1.29 (IO5)
- new net FLASH_CS: R31.2, U1.37 (IO23), U3.1 (~{CS})
- new net Relay Driver4/Relay+: J8.2 (Pin_2)
- new net Relay Driver4/Relay-: J8.1 (Pin_1)
- new net Relay Driver5/Relay+: J9.2 (Pin_2)
- new net Relay Driver5/Relay-: J9.1 (Pin_1)
- new net SPI_CLK: U1.31 (IO19), U3.6 (CLK)
- new net SPI_MISO: U1.33 (IO21), U3.2 (DO/IO_{1})
- new net SPI_MOSI: U1.30 (IO18), U3.5 (DI/IO_{0})
- new net UART0_RX: J11.3 (Pin_3), U1.34 (RXD0/IO3)
- new net UART0_TX: J11.2 (Pin_2), U1.35 (TXD0/IO1)
- no-connect marks 23 -> 8
Other:
- sheet 5V Power Converter renamed Power Supply
- added sheet Relay Driver4 (Relay Driver.kicad_sch)
- added sheet Relay Driver5 (Relay Driver.kicad_sch)
- moved on the sheet: C10, C9, D17, D18, J4, J5, R24
