File: Furnace_Controller_V1/Relay Driver.kicad_sch (KiCad schematic)
At the start: 8 parts, among them Q1 IRLZ44N

Commit message: V2 dev
Parts:
- removed D2: 1N4148, Diode_THT:D_DO-35_SOD27_P7.62mm_Horizontal, symbol Diode:1N4148
- removed TP7: LGND_TP, TestPoint:TestPoint_Pad_D1.5mm, symbol Connector:TestPoint
- added D16: SM4007, Diode_SMD:D_SOD-123, symbol Diode:SM4007
- D6: footprint LED_SMD:LED_0805_2012Metric -> LED_SMD:LED_0603_1608Metric
- Q1: value IRLZ44N -> HL3402; footprint Package_TO_SOT_THT:TO-220-3_Vertical -> Package_TO_SOT_SMD:TSOT-23
- R12, R4, R5: footprint Resistor_SMD:R_0805_2012Metric_Pad1.20x1.40mm_HandSolder -> Resistor_SMD:R_0603_1608Metric
- TP3: footprint TestPoint:TestPoint_Pad_D1.5mm -> TestPoint:TestPoint_Pad_D1.0mm
Connections:
- net Relay_GND is gone; now on net Logic_GND: Q1.3 (S)
- net +24V: now also D16.1 (K)
- net Relay-: now also D16.2 (A)
