File: Furnace_Controller_V1/nextion_level_shifter.kicad_sch (KiCad schematic)
At the start: 20 parts, among them U4 TXU0101DBVR, U5 TXU0101DBVR

Commit message: V2 dev
Parts:
- removed TP20: 5V_TP, TestPoint:TestPoint_Pad_D1.5mm, symbol Connector:TestPoint
- removed TP21: 3V3_TP, TestPoint:TestPoint_Pad_D1.5mm, symbol Connector:TestPoint
- C5, C6, C7, C8: footprint Capacitor_SMD:C_0805_2012Metric_Pad1.18x1.45mm_HandSolder -> Capacitor_SMD:C_0603_1608Metric
- D12, D13, D14, D15: footprint LED_SMD:LED_0805_2012Metric -> LED_SMD:LED_0603_1608Metric
- R20, R21, R22, R23: footprint Resistor_SMD:R_0805_2012Metric_Pad1.20x1.40mm_HandSolder -> Resistor_SMD:R_0603_1608Metric
- TP22, TP23, TP24, TP25: footprint TestPoint:TestPoint_Pad_D1.5mm -> TestPoint:TestPoint_Pad_D1.0mm
Connections:
- net +3.3V renamed +3V3
