File: Furnace_Controller_V2/Furnace_Controller.kicad_pcb (KiCad board)
At the start: 2 copper layers, 149 x 141 mm, 99 parts, among them J1 Power In Treminal, J3 Relay Terminal, J4 HMD Terminal, J5 RS-485 Terminal, Q1 IRLZ44N, Q2 IRLZ44N, Q3 IRLZ44N, Q4 IRLZ44N, Q5 2n2222, U2 LM2596S-5, U3 THVD2450DR, U4 TXU0101DBVR, U5 TXU0101DBVR, U6 TVS3300DRV

Commit message: Organize PCB revisions and correct TI footprints
Parts:
- removed C6: 100n, Capacitor_SMD:C_0805_2012Metric_Pad1.18x1.45mm_HandSolder
- removed D1, D16: 1N5822, Diode_THT:D_DO-201AD_P15.24mm_Horizontal
- removed D13, D14, D15, D3: LED, LED_SMD:LED_0805_2012Metric
- removed D17, D18: SMAJ30CA, Diode_SMD:D_SMA
- removed D19, D2, D4: 1N4148, Diode_THT:D_DO-35_SOD27_P7.62mm_Horizontal
- removed F2: 3588, MiniAutoFuse:3588
- removed H2: MountingHole, MountingHole:MountingHole_5.3mm_M5
- removed R10: 100, Resistor_SMD:R_0805_2012Metric_Pad1.20x1.40mm_HandSolder
- removed R9: 68, Resistor_SMD:R_0805_2012Metric_Pad1.20x1.40mm_HandSolder
- removed TP1, TP3, TP4, TP6: HR_TP, TestPoint:TestPoint_Pad_D1.5mm
- removed TP11, TP5, TP7, TP8, TP9: LGND_TP, TestPoint:TestPoint_Pad_D1.5mm
- removed TP12: RSB_TP, TestPoint:TestPoint_Pad_D1.5mm
- removed TP13: RSA_TP, TestPoint:TestPoint_Pad_D1.5mm
- removed TP14, TP20: 5V_TP, TestPoint:TestPoint_Pad_D1.5mm
- removed TP15: U2RX_TP, TestPoint:TestPoint_Pad_D1.5mm
- removed TP16: U2TX_TP, TestPoint:TestPoint_Pad_D1.5mm
- removed TP18: RS_DIR, TestPoint:TestPoint_Pad_D1.5mm
- removed TP19, TP21: 3V3_TP, TestPoint:TestPoint_Pad_D1.5mm
- removed TP2: PGND_TP, TestPoint:TestPoint_Pad_D1.5mm
- removed TP22: U1TX_TP, TestPoint:TestPoint_Pad_D1.5mm
- removed TP23: U1RX_TP, TestPoint:TestPoint_Pad_D1.5mm
- removed TP24: HMDTX_TP, TestPoint:TestPoint_Pad_D1.5mm
- removed TP25: HMDRX_TP, TestPoint:TestPoint_Pad_D1.5mm
- removed TP26: 24V_TP, TestPoint:TestPoint_Pad_D1.5mm
- removed U2: LM2596S-5, Package_TO_SOT_SMD:TO-263-5_TabPin3
- removed U3: THVD2450DR, THVD:SOIC127P600X175-8N
- added C11: 1u, Capacitor_SMD:C_0603_1608Metric, F.Cu at (160.6, 113.5)
- added C12: 1u, Capacitor_SMD:C_0603_1608Metric, F.Cu at (155.4, 106.7)
- added C13: 100n, Capacitor_SMD:C_0603_1608Metric, F.Cu at (161.8, 104.1)
- added C14: 1n, Capacitor_SMD:C_1808_4520Metric, F.Cu at (165.6, 112.8)
- added C15: 1u, Capacitor_SMD:C_0603_1608Metric, F.Cu at (163.3, 104.2)
- added C16: 470p, Capacitor_SMD:C_0603_1608Metric, F.Cu at (162.0, 97.4)
- added C17: 1u, Capacitor_SMD:C_0603_1608Metric, F.Cu at (162.0, 98.9)
- added C18: 100n, Capacitor_SMD:C_0603_1608Metric, F.Cu at (157.1, 96.1)
- added C19: 1u, Capacitor_SMD:C_0603_1608Metric, F.Cu at (155.5, 96.1)
- added C20: 1u, Capacitor_SMD:C_0603_1608Metric, F.Cu at (148.1, 111.0)
- added C21: 100n, Capacitor_SMD:C_0603_1608Metric, F.Cu at (148.1, 109.4)
- added C22: 100n, Capacitor_SMD:C_0603_1608Metric, F.Cu at (149.3, 104.4)
- added C23: 1u, Capacitor_SMD:C_0603_1608Metric, F.Cu at (149.3, 102.9)
- added C24: 100n, Capacitor_SMD:C_0603_1608Metric, F.Cu at (205.7, 114.2)
- added C25: 1u, Capacitor_SMD:C_0603_1608Metric, F.Cu at (262.4, 104.4)
- added C26: 100n, Capacitor_SMD:C_0603_1608Metric, F.Cu at (262.4, 106.9)
- added C27: 100n, Capacitor_SMD:C_0603_1608Metric, F.Cu at (262.4, 109.4)
- added C28: 1u, Capacitor_SMD:C_0603_1608Metric, F.Cu at (262.4, 111.9)
- added C29: 47u, Capacitor_THT:CP_Radial_D6.3mm_P2.50mm, F.Cu at (149.0, 81.8)
- added C30: 2.2u, Capacitor_SMD:C_0603_1608Metric, F.Cu at (152.7, 80.7)
- added C31: 100n, Capacitor_SMD:C_0603_1608Metric, F.Cu at (152.7, 79.2)
- added C32: 10n, Capacitor_SMD:C_0603_1608Metric, F.Cu at (152.7, 68.7)
- added C33: 100n, Capacitor_SMD:C_0603_1608Metric, F.Cu at (149.7, 77.7)
- added C34: 47u, Capacitor_THT:CP_Radial_D6.3mm_P2.50mm, F.Cu at (138.9, 79.8)
- added C35: 10u, Capacitor_SMD:C_0805_2012Metric, F.Cu at (139.7, 75.2)
- added C36: 100n, Capacitor_SMD:C_0603_1608Metric, F.Cu at (139.7, 73.5)
- added C37: 100n, Capacitor_SMD:C_0603_1608Metric, F.Cu at (197.2, 100.8)
- added C38: 100n, Capacitor_SMD:C_0603_1608Metric, F.Cu at (239.4, 118.5)
- added C39: 10u, Capacitor_SMD:C_0805_2012Metric, F.Cu at (243.6, 129.1)
- added C40: 100n, Capacitor_SMD:C_0603_1608Metric, F.Cu at (239.4, 121.0)
- added C41: 10u, Capacitor_SMD:C_0805_2012Metric, F.Cu at (243.6, 132.2)
- added FB1: FerriteBead, Inductor_SMD:L_0603_1608Metric, F.Cu at (157.1, 113.5)
- added H5: MountingHole, MountingHole:MountingHole_2.2mm_M2, F.Cu at (135.4, 66.2)
- added H6: MountingHole, MountingHole:MountingHole_3.2mm_M3, F.Cu at (137.0, 132.7)
- added J2: Power In Treminal, Connector_Phoenix_MC:PhoenixContact_MC_1,5_2-G-3.5_1x02_P3.50mm_Horizontal, F.Cu at (140.3, 90.2)
- added J6: Relay Terminal, Connector_Phoenix_MC:PhoenixContact_MC_1,5_2-G-3.5_1x02_P3.50mm_Horizontal, F.Cu at (185.2, 128.6)
- added J7: Relay Terminal, Connector_Phoenix_MC:PhoenixContact_MC_1,5_2-G-3.5_1x02_P3.50mm_Horizontal, F.Cu at (175.6, 128.6)
- added J8: Relay Terminal, Connector_Phoenix_MC:PhoenixContact_MC_1,5_2-G-3.5_1x02_P3.50mm_Horizontal, F.Cu at (204.6, 128.6)
- added J9: RJ45_Bel_SI-60062-F, Connector_RJ:RJ45_Bel_SI-60062-F, F.Cu at (154.6, 119.4)
- added JP1: Jumper_2_Open, TestPoint:TestPoint_2Pads_Pitch2.54mm_Drill0.8mm, F.Cu at (144.2, 99.3)
- added JP2: Jumper_2_Open, TestPoint:TestPoint_2Pads_Pitch2.54mm_Drill0.8mm, F.Cu at (144.1, 102.9)
- added R2: 10k, Resistor_SMD:R_0603_1608Metric, F.Cu at (189.0, 106.8)
- added R26: 10k, Resistor_SMD:R_0603_1608Metric, F.Cu at (199.3, 120.3)
- added R27: 100, Resistor_SMD:R_0603_1608Metric, F.Cu at (191.3, 120.3)
- added R28: 10k, Resistor_SMD:R_0603_1608Metric, F.Cu at (189.7, 120.3)
- added R29: 100, Resistor_SMD:R_0603_1608Metric, F.Cu at (175.6, 122.5)
- added R30: 10k, Resistor_SMD:R_0603_1608Metric, F.Cu at (170.7, 120.8)
- added R31: 100, Resistor_SMD:R_0603_1608Metric, F.Cu at (208.6, 121.9)
- added R32: 10k, Resistor_SMD:R_0603_1608Metric, F.Cu at (210.2, 121.9)
- added R33: 56k, Resistor_SMD:R_0603_1608Metric, F.Cu at (156.0, 74.8)
- added R34: 100k, Resistor_SMD:R_0603_1608Metric, F.Cu at (152.7, 77.7)
- added R35: 56k, Resistor_SMD:R_0603_1608Metric, F.Cu at (152.7, 65.6)
- added R36: 10k, Resistor_SMD:R_0603_1608Metric, F.Cu at (152.7, 67.1)
- added R37: 15, Resistor_SMD:R_0603_1608Metric, F.Cu at (201.0, 103.4)
- added R38: 15, Resistor_SMD:R_0603_1608Metric, F.Cu at (201.0, 105.0)
- added R39: 100, Resistor_SMD:R_0603_1608Metric, F.Cu at (193.5, 108.8)
- added R40: 100, Resistor_SMD:R_0603_1608Metric, F.Cu at (193.6, 110.5)
- added R41: 10k, Resistor_SMD:R_0603_1608Metric, F.Cu at (239.4, 123.6)
- added R42: 10k, Resistor_SMD:R_0603_1608Metric, F.Cu at (239.4, 126.1)
- added R43: 10k, Resistor_SMD:R_0603_1608Metric, F.Cu at (239.4, 128.6)
- added R44: 0, Resistor_SMD:R_0603_1608Metric, F.Cu at (239.4, 131.1)
- added SW1: SW_Push, Button_Switch_THT:SW_PUSH_6mm_H4.3mm, F.Cu at (138.2, 118.0)
- added U10: PTHVD2452VDR, PCM_JLCPCB:SOIC-14_L8.7-W3.9-P1.27-LS6.0-BL, F.Cu at (245.6, 122.5)
- added U11: TPS36BA38ACADDFRQ1, Furnace_TI:SOT-23-THIN-8_DDF_TEX, F.Cu at (258.3, 119.7)
- added U7: TPS7A20xxxDBV, Package_TO_SOT_SMD:SOT-23-5, F.Cu at (267.0, 105.5)
- added U8: LMR16030SDDAR, Package_SO:SOIC-8-1EP_3.9x4.9mm_P1.27mm_EP2.29x3mm, F.Cu at (152.4, 73.1)
- added U9: THVD2450DR, PCM_JLCPCB:SOIC-8_3.9x4.9mm_P1.27mm, F.Cu at (195.3, 104.2)
- added Y1: Crystal_GND24, Crystal:Crystal_SMD_3225-4Pin_3.2x2.5mm, F.Cu at (168.3, 99.7)
- C1: value 220u -> 100n; footprint Capacitor_THT:CP_Radial_D12.5mm_P5.00mm -> Capacitor_SMD:C_0603_1608Metric
- C10: value 10u -> 100n; footprint Capacitor_THT:CP_Radial_D5.0mm_P2.00mm -> Capacitor_SMD:C_0603_1608Metric
- C2: value 100n -> 10u; footprint Capacitor_SMD:C_0805_2012Metric_Pad1.18x1.45mm_HandSolder -> Capacitor_SMD:C_0805_2012Metric
- C3: value 47u -> 100n; footprint Capacitor_THT:CP_Radial_D8.0mm_P2.50mm -> Capacitor_SMD:C_0603_1608Metric
- C4: value 10u -> 3.3n; footprint Capacitor_THT:CP_Radial_D5.0mm_P2.00mm -> Capacitor_SMD:C_0603_1608Metric
- C5: value 100n -> 22n; footprint Capacitor_SMD:C_0805_2012Metric_Pad1.18x1.45mm_HandSolder -> Capacitor_SMD:C_0603_1608Metric
- C7, C8: value 100n -> 18p; footprint Capacitor_SMD:C_0805_2012Metric_Pad1.18x1.45mm_HandSolder -> Capacitor_SMD:C_0603_1608Metric
- C9: value 100n -> 10n; footprint Capacitor_SMD:C_0805_2012Metric_Pad1.18x1.45mm_HandSolder -> Capacitor_SMD:C_0603_1608Metric
- D10: value LED -> SS36; footprint LED_SMD:LED_0805_2012Metric -> Diode_SMD:D_SMA
- D11: value LED -> SM712_SOT23; footprint LED_SMD:LED_0805_2012Metric -> Package_TO_SOT_SMD:SOT-23
- D12: value LED -> SS14; footprint LED_SMD:LED_0805_2012Metric -> Diode_SMD:D_SOD-123
- D5, D6, D8: value LED -> SM4007; footprint LED_SMD:LED_0805_2012Metric -> Diode_SMD:D_SOD-123
- D7: value 1N4148 -> SM4007; footprint Diode_THT:D_DO-35_SOD27_P7.62mm_Horizontal -> Diode_SMD:D_SOD-123
- D9: value 1N4148 -> SS36; footprint Diode_THT:D_DO-35_SOD27_P7.62mm_Horizontal -> Diode_SMD:D_SMA
- H1, H3, H4: footprint MountingHole:MountingHole_5.3mm_M5 -> MountingHole:MountingHole_3.2mm_M3
- J1: value Power In Treminal -> Conn_01x04_Socket; footprint TerminalBlock:TerminalBlock_MaiXu_MX126-5.0-02P_1x02_P5.00mm -> Connector_PinHeader_2.54mm:PinHeader_1x04_P2.54mm_Vertical
- J3: value Relay Terminal -> Screw_Terminal_01x05; footprint TerminalBlock:TerminalBlock_MaiXu_MX126-5.0-09P_1x09_P5.00mm -> Connector_Phoenix_MC:PhoenixContact_MC_1,5_5-G-3.5_1x05_P3.50mm_Horizontal
- J4: value HMD Terminal -> RS-485-Terminal; footprint TerminalBlock:TerminalBlock_MaiXu_MX126-5.0-04P_1x04_P5.00mm -> Connector_Phoenix_MC:PhoenixContact_MC_1,5_3-G-3.5_1x03_P3.50mm_Horizontal
- J5: value RS-485 Terminal -> Relay Terminal; footprint TerminalBlock:TerminalBlock_MaiXu_MX126-5.0-04P_1x04_P5.00mm -> Connector_Phoenix_MC:PhoenixContact_MC_1,5_2-G-3.5_1x02_P3.50mm_Horizontal
- L1: footprint Coil:SRR1260-150M -> Inductor_SMD:L_6.3x6.3_H3
- Q1, Q2, Q3, Q4: value IRLZ44N -> 20N04-MS; footprint Package_TO_SOT_THT:TO-220-3_Vertical -> PCM_JLCPCB:Q_SOT-89
- Q5: value 2n2222 -> HL3402; footprint Package_TO_SOT_THT:TO-92_Inline -> PCM_JLCPCB:Q_SOT-23
- R1, R3: footprint Resistor_SMD:R_0805_2012Metric_Pad1.20x1.40mm_HandSolder -> Resistor_SMD:R_0603_1608Metric
- R11, R15, R5, R8: value 47k -> 10k; footprint Resistor_SMD:R_0805_2012Metric_Pad1.20x1.40mm_HandSolder -> Resistor_SMD:R_0603_1608Metric
- R12, R13, R19: value 68 -> 10k; footprint Resistor_SMD:R_0805_2012Metric_Pad1.20x1.40mm_HandSolder -> Resistor_SMD:R_0603_1608Metric
- R14, R4, R7: value 100 -> 10k; footprint Resistor_SMD:R_0805_2012Metric_Pad1.20x1.40mm_HandSolder -> Resistor_SMD:R_0603_1608Metric
- R16: value 15 -> 10k; footprint Resistor_SMD:R_0805_2012Metric_Pad1.20x1.40mm_HandSolder -> Resistor_SMD:R_0603_1608Metric
- R17: value 15 -> 330; footprint Resistor_SMD:R_0805_2012Metric_Pad1.20x1.40mm_HandSolder -> Resistor_SMD:R_0603_1608Metric
- R18, R22: value 68 -> 49.9; footprint Resistor_SMD:R_0805_2012Metric_Pad1.20x1.40mm_HandSolder -> Resistor_SMD:R_0603_1608Metric
- R20: value 330 -> 49.9; footprint Resistor_SMD:R_0805_2012Metric_Pad1.20x1.40mm_HandSolder -> Resistor_SMD:R_0603_1608Metric
- R21: value 68 -> 330; footprint Resistor_SMD:R_0805_2012Metric_Pad1.20x1.40mm_HandSolder -> Resistor_SMD:R_0603_1608Metric
- R23: value 330 -> 12,1k; footprint Resistor_SMD:R_0805_2012Metric_Pad1.20x1.40mm_HandSolder -> Resistor_SMD:R_0603_1608Metric
- R24: value 120 -> 49.9; footprint Resistor_SMD:R_0805_2012Metric_Pad1.20x1.40mm_HandSolder -> Resistor_SMD:R_0603_1608Metric
- R25: value 1k -> 100; footprint Resistor_SMD:R_0805_2012Metric_Pad1.20x1.40mm_HandSolder -> Resistor_SMD:R_0603_1608Metric
- R6: value 68 -> 120; footprint Resistor_SMD:R_0805_2012Metric_Pad1.20x1.40mm_HandSolder -> Resistor_SMD:R_0603_1608Metric
- U1: value ~ -> ESP32-WROOM-32E-N8; footprint Custom_Footprints:ESP32_DevKitc_V4 -> RF_Module:ESP32-WROOM-32
- U4: value TXU0101DBVR -> LAN8720A; footprint TXU:SOT95P280X145-6N -> Package_DFN_QFN:VQFN-24-1EP_4x4mm_P0.5mm_EP2.5x2.5mm_ThermalVias
- U5: value TXU0101DBVR -> TPS7A20xxxDBV; footprint TXU:SOT95P280X145-6N -> Package_TO_SOT_SMD:SOT-23-5
- U6: value TVS3300DRV -> TCA9534; footprint Package_SON:WSON-6-1EP_2x2mm_P0.65mm_EP1x1.6mm -> Package_SO:TSSOP-16_4.4x5mm_P0.65mm
- moved C3 200.2 mm to (253.8, 118.5), turned to 0 degrees
- moved H3 189.4 mm to (214.8, 132.9)
- moved U6 145.4 mm to (200.9, 115.5)
- moved C1 138.1 mm to (170.3, 86.6), turned to 90 degrees
- moved R7 134.4 mm to (253.8, 126.1)
- moved R8 131.6 mm to (253.8, 128.6), turned to 0 degrees
- moved C4 120.9 mm to (253.8, 121.0), turned to 0 degrees
- moved C5 118.2 mm to (253.8, 123.6), turned to 0 degrees
- moved R25 114.6 mm to (200.9, 120.3), turned to -90 degrees
- moved BZ1 111.5 mm to (176.9, 109.7)
- moved Q5 111.2 mm to (194.0, 113.2), turned to 0 degrees
- moved H1 108.1 mm to (116.5, 84.3)
- moved L1 104.6 mm to (142.0, 69.2)
- moved D8 104.5 mm to (206.4, 124.8), turned to 180 degrees
- moved J1 103.4 mm to (138.4, 107.0)
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Connections:
- C1 pad 1: +5V -> +3.3V
- C1 pad 2: Logic_GND -> GND
- C10 pad 1: +5V -> +3.3VA
- C10 pad 2: Logic_GND -> GND
- C2 pad 2: Logic_GND -> GND
- C3 pad 1: +24V -> +3.3V
- C3 pad 2: Logic_GND -> GND
- C4 pad 1: +3.3V -> Net-(U11-CWS)
- C4 pad 2: Logic_GND -> GND
- C5 pad 1: +3.3V -> Net-(U11-CRST)
- C5 pad 2: Logic_GND -> GND
- C7 pad 1: +5V -> GND
- C7 pad 2: Logic_GND -> Net-(U4-XTAL1/CLKIN)
- C8 pad 1: +3.3V -> Net-(U4-XTAL2)
- C8 pad 2: Logic_GND -> GND
- C9 pad 1: +5V -> Net-(J9-RCT)
- C9 pad 2: Logic_GND -> GND
- D10 pad 2: /UART2_TX -> GND
- D11 pad 1: Net-(D11-K) -> /rs485-module/B
- D11 pad 2: /UART2_RX -> /rs485-module/A
- D12 pad 1: Net-(D12-K) -> Net-(BZ1--)
- D12 pad 2: /Nextion Level Shifter/HMD_TX -> +5V
- D5 pad 1: Net-(D5-K) -> +24V
- D5 pad 2: /Aux2_Relay_Pin -> /Relay Driver/Relay-
- D6 pad 1: Net-(D6-K) -> +24V
- D6 pad 2: /Heater_Relay_Pin -> /Relay Driver1/Relay-
- D7 pad 2: /Relay Driver3/Relay- -> /Relay Driver2/Relay-
- D8 pad 1: Net-(D8-K) -> +24V
- D8 pad 2: /Fan_Relay_Pin -> /Relay Driver3/Relay-
- D9 pad 1: +24V -> Net-(D9-K)
- D9 pad 2: /Relay Driver1/Relay- -> +24V
- J1 pad 1: Logic_GND -> GND
- J1 pad 2: /5V Power Converter/Power In -> /UART0_RX
- J3 pad 1: Relay_GND -> GND
- J3 pad 2: /Relay Driver3/Relay- -> /RS-422-module/Y
- J3 pad 3: +24V -> /RS-422-module/Z
- J3 pad 4: /Relay Driver2/Relay- -> /RS-422-module/B
- J3 pad 5: +24V -> /RS-422-module/A
- J4 pad 1: Logic_GND -> GND
- J4 pad 2: /Nextion Level Shifter/HMD_TX -> /rs485-module/A
- J4 pad 3: /Nextion Level Shifter/HMD_RX -> /rs485-module/B
- J5 pad 1: Logic_GND -> /Relay Driver/Relay-
- J5 pad 2: /RS-485 Transeiver/RS-485_A -> +24V
- L1 pad 1: Net-(D1-K) -> Net-(D10-K)
- Q1 pad 3: Relay_GND -> GND
- Q2 pad 2: /Relay Driver2/Relay- -> /Relay Driver1/Relay-
- Q2 pad 3: Relay_GND -> GND
- Q3 pad 2: /Relay Driver3/Relay- -> /Relay Driver2/Relay-
- Q3 pad 3: Relay_GND -> GND
- Q4 pad 2: /Relay Driver1/Relay- -> /Relay Driver3/Relay-
- Q4 pad 3: Relay_GND -> GND
- Q5 pad 1: Net-(BZ1--) -> Net-(Q5-G)
- Q5 pad 2: Net-(Q5-B) -> Net-(BZ1--)
- Q5 pad 3: Logic_GND -> GND
- R1 pad 2: /UART2_RX -> /*RESET
- R11 pad 1: Net-(Q3-G) -> +3.3V
- R11 pad 2: Logic_GND -> /~{RST}
- R12 pad 1: Net-(D6-K) -> +3.3V
- R12 pad 2: Logic_GND -> /CRS_DV
- R13 pad 1: Net-(D8-K) -> +3.3V
- R13 pad 2: Logic_GND -> Net-(U4-RXER/PHYAD0)
- R14 pad 1: /Fan_Relay_Pin -> +3.3V
- R14 pad 2: Net-(Q4-G) -> /RXD1
- R15 pad 1: Net-(Q4-G) -> +3.3V
- R15 pad 2: Logic_GND -> /RXD0
- R16 pad 1: /RS-485 Transeiver/RS-485_B -> Net-(U4-LED2/~{INTSEL})
- R16 pad 2: Net-(U3-B) -> GND
- R17 pad 1: /RS-485 Transeiver/RS-485_A -> Net-(U4-LED2/~{INTSEL})
- R17 pad 2: Net-(U3-A) -> /Ethernet Module/NET_LED_G_A
- R18 pad 1: Net-(D10-K) -> Net-(J9-RCT)
- R18 pad 2: Logic_GND -> Net-(J9-TD+)
- R19 pad 1: Net-(D11-K) -> Net-(U4-LED1/REGOFF)
- R19 pad 2: Logic_GND -> GND
- R20 pad 1: Net-(D12-K) -> Net-(J9-RCT)
- R20 pad 2: Logic_GND -> Net-(J9-TD-)
- R21 pad 1: Net-(D13-K) -> Net-(U4-LED1/REGOFF)
- R21 pad 2: Logic_GND -> /Ethernet Module/NET_LED_Y_A
- R22 pad 1: Net-(D14-K) -> Net-(J9-RCT)
- R22 pad 2: Logic_GND -> Net-(J9-RD+)
- R23 pad 1: Net-(D15-K) -> Net-(U4-RBIAS)
- R23 pad 2: Logic_GND -> GND
- R24 pad 1: /RS-485 Transeiver/RS-485_B -> Net-(J9-RCT)
- R24 pad 2: /RS-485 Transeiver/RS-485_A -> Net-(J9-RD-)
- R25 pad 1: Net-(U1-GPIO23) -> /Heater_Relay_Pin
- R25 pad 2: Net-(Q5-B) -> Net-(Q1-G)
- R3 pad 1: /RS_485_DIR -> /WDI
- R3 pad 2: Logic_GND -> GND
- R4 pad 1: /Heater_Relay_Pin -> +3.3V
- R4 pad 2: Net-(Q1-G) -> /SCL
- R5 pad 1: Net-(Q1-G) -> +3.3V
- R5 pad 2: Logic_GND -> Net-(U1-IO12)
- R6 pad 1: Net-(D3-K) -> /rs485-module/B
- R6 pad 2: Logic_GND -> /rs485-module/A
- R7 pad 1: /Aux_Relay_Pin -> Net-(U11-SET1)
- R7 pad 2: Net-(Q2-G) -> GND
- R8 pad 1: Net-(Q2-G) -> Net-(U11-SET0)
- R8 pad 2: Logic_GND -> GND
- U1 pad 1: +3.3V -> GND
- U1 pad 10: /UART2_RX -> /RXD0
- U1 pad 11: /UART2_TX -> /RXD1
- U1 pad 12: unconnected-(U1-GPIO14-Pad12) -> /CRS_DV
- U1 pad 13: unconnected-(U1-GPIO12-Pad13) -> /MDC
- U1 pad 14: Logic_GND -> Net-(U1-IO12)
- U1 pad 15: unconnected-(U1-GPIO13-Pad15) -> GND
- U1 pad 16: unconnected-(U1-GPIO9-Pad16) -> /MDIO
- U1 pad 19: +5V -> unconnected-(U1-SCS/CMD-Pad19)
- U1 pad 2: unconnected-(U1-EN-Pad2) -> +3.3V
- U1 pad 23: unconnected-(U1-GPIO15-Pad23) -> /WDI
- U1 pad 24: unconnected-(U1-GPIO2-Pad24) -> /SCL
- U1 pad 25: unconnected-(U1-GPIO0-Pad25) -> /REFCLKO
- U1 pad 26: unconnected-(U1-GPIO4-Pad26) -> /UART2_TX
- U1 pad 27: /UART1_RX -> /RS_485_DIR
- U1 pad 28: /UART1_TX -> /UART2_RX
- U1 pad 29: unconnected-(U1-GPIO5-Pad29) -> /BUZZER
- U1 pad 3: unconnected-(U1-GPIO36-Pad3) -> /*RESET
- U1 pad 30: /Aux2_Relay_Pin -> /UART1_RX
- U1 pad 31: /Aux_Relay_Pin -> /TXD0
- U1 pad 32: Logic_GND -> unconnected-(U1-NC-Pad32)
- U1 pad 33: /Fan_Relay_Pin -> /TXEN
- U1 pad 34: unconnected-(U1-GPIO3/U0RXD-Pad34) -> /UART0_RX
- U1 pad 35: unconnected-(U1-GPIO1/U0TXD-Pad35) -> /UART0_TX
- U1 pad 36: /Heater_Relay_Pin -> /TXD1
- U1 pad 37: Net-(U1-GPIO23) -> /UART1_TX
- U1 pad 38: Logic_GND -> GND
- U1 pad 8: unconnected-(U1-GPIO33-Pad8) -> /SDA
- U1 pad 9: /RS_485_DIR -> /~{RST}
- U4 pad 1: +5V -> +3.3VA
- U4 pad 2: Logic_GND -> Net-(U4-LED2/~{INTSEL})
- U4 pad 3: /Nextion Level Shifter/HMD_TX -> Net-(U4-LED1/REGOFF)
- U4 pad 4: /UART1_RX -> Net-(U4-XTAL2)
- U4 pad 5: +3.3V -> Net-(U4-XTAL1/CLKIN)
- U4 pad 6: +3.3V -> /Ethernet Module/VDDCR
- U5 pad 1: +3.3V -> +5V
- U5 pad 2: Logic_GND -> GND
- U5 pad 3: /UART1_TX -> +5V
- U5 pad 4: /Nextion Level Shifter/HMD_RX -> unconnected-(U5-NC-Pad4)
- U5 pad 5: +5V -> +3.3VA
- U6 pad 1: Logic_GND -> unconnected-(U6-A0-Pad1)
- U6 pad 2: Logic_GND -> unconnected-(U6-A1-Pad2)
- U6 pad 3: Logic_GND -> unconnected-(U6-A2-Pad3)
- U6 pad 4: +24V -> /Heater_Relay_Pin
- U6 pad 5: +24V -> /Fan_Relay_Pin
- U6 pad 6: +24V -> /Aux_Relay_Pin
- U6 pad 7: Logic_GND -> /Aux2_Relay_Pin
Routing:
- net +5V: track 295.2 -> 118.9 mm, vias 1 -> 3
- net +24V: track 294.7 -> 158.4 mm
- net /RS_485_DIR: track 97.2 -> 6.77 mm
- net /UART2_TX: track 93.4 -> 7.21 mm
- net /UART2_RX: track 89.6 -> 5.76 mm
- net Net-(U1-GPIO23): track 65.3 -> 0.00 mm, vias 1 -> 0
- net Net-(U4-LED1/REGOFF): track 0.00 -> 65.2 mm, vias 0 -> 2
- net /UART1_RX: track 60.4 -> 0.00 mm
- net Relay_GND: track 60.1 -> 0.00 mm
- net /UART1_TX: track 57.4 -> 0.00 mm
- net /UART0_RX: track 0.00 -> 57.3 mm, vias 0 -> 1
- net /UART0_TX: track 0.00 -> 56.4 mm, vias 0 -> 1
- net /REFCLKO: track 0.00 -> 55.2 mm, vias 0 -> 3
- net /TXD1: track 0.00 -> 49.4 mm, vias 0 -> 2
- net /TXD0: track 0.00 -> 46.7 mm, vias 0 -> 2
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- added copper zone on B.Cu, net GND
- added copper zone on F.Cu, net GND
- added copper zone on In1.Cu, net GND
- added copper zone on In2.Cu, net GND
- removed copper zone on B.Cu, net Logic_GND
- removed copper zone on F.Cu, net Logic_GND
Other:
- board size 149 x 141 mm -> 85.6 x 72.7 mm
- copper layers 2 -> 4
- board text added: "3V3"
- board text added: "3V3 EN"
- board text added: "BOOT"
- board text added: "BOOT EN"
- board text added: "Designed in Bulgaria"
- board text added: "GND"
- board text added: "TM_FC_4R_V2"
- board text added: "U0RX"
- board text added: "U0TX"
- board text removed: "V1.0P"
- board text removed: "VT KA SK"

Commit message: Normalize 3.3V net names
Connections:
- net +3.3V renamed +3V3
- net +3.3VA renamed +3V3A
