File: Furnace_Controller_V1/sheets/rs-485_transeiver.kicad_sch (KiCad schematic)
At the start: 18 parts, among them U3 THVD2450DR

Commit message: Normalize 3.3V net names
Connections:
- net +3.3V renamed +3V3
Changed lines of the file:
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@@
 	)
 	(symbol
-		(lib_id "power:+3.3V")
+		(lib_id "power:+3V3")
 		(at 196.85 72.39 0)
 		(unit 1)
@@
 			)
 		)
-		(property "Value" "+3.3V"
+		(property "Value" "+3V3"
 			(at 196.85 67.31 0)
 			(effects
@@
 			)
 		)
-		(property "Description" "Power symbol creates a global label with name \"+3.3V\""
+		(property "Description" "Power symbol creates a global label with name \"+3V3\""
 			(at 196.85 72.39 0)
 			(effects
@@
 	)
 	(symbol
-		(lib_id "power:+3.3V")
+		(lib_id "power:+3V3")
 		(at 165.1 69.85 0)
 		(unit 1)
@@
 			)
 		)
-		(property "Value" "+3.3V"
+		(property "Value" "+3V3"
 			(at 165.1 64.77 0)
 			(effects
@@
 			)
 		)
-		(property "Description" "Power symbol creates a global label with name \"+3.3V\""
+		(property "Description" "Power symbol creates a global label with name \"+3V3\""
 			(at 165.1 69.85 0)
 			(effects
@@
 	)
 	(symbol
-		(lib_id "power:+3.3V")
+		(lib_id "power:+3V3")
 		(at 118.11 63.5 0)
 		(unit 1)
@@
 			)
 		)
-		(property "Value" "+3.3V"
+		(property "Value" "+3V3"
 			(at 118.11 58.42 0)
 			(effects
@@
 			)
 		)
-		(property "Description" "Power symbol creates a global label with name \"+3.3V\""
+		(property "Description" "Power symbol creates a global label with name \"+3V3\""
 			(at 118.11 63.5 0)
 			(effects
