File: Furnace_Controller_V2/sheets/ethernet_module.kicad_sch (KiCad schematic)
At the start: 31 parts, among them J9 RJ45_Bel_SI-60062-F, U4 LAN8720A, Y1 Crystal_GND24

Commit message: Normalize 3.3V net names
Connections:
- net +3.3V renamed +3V3
- net +3.3VA renamed +3V3A
Changed lines of the file:
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@@
 	)
 	(symbol
-		(lib_id "power:+3.3V")
+		(lib_id "power:+3V3")
 		(at 104.14 40.64 0)
 		(unit 1)
@@
 			)
 		)
-		(property "Value" "+3.3V"
+		(property "Value" "+3V3"
 			(at 104.14 35.56 0)
 			(show_name no)
@@
 			)
 		)
-		(property "Description" "Power symbol creates a global label with name \"+3.3V\""
+		(property "Description" "Power symbol creates a global label with name \"+3V3\""
 			(at 104.14 40.64 0)
 			(hide yes)
@@
 	)
 	(symbol
-		(lib_id "power:+3.3V")
+		(lib_id "power:+3V3")
 		(at 26.67 57.15 0)
 		(unit 1)
@@
 			)
 		)
-		(property "Value" "+3.3V"
+		(property "Value" "+3V3"
 			(at 26.67 52.07 0)
 			(show_name no)
@@
 			)
 		)
-		(property "Description" "Power symbol creates a global label with name \"+3.3V\""
+		(property "Description" "Power symbol creates a global label with name \"+3V3\""
 			(at 26.67 57.15 0)
 			(hide yes)
@@
 	)
 	(symbol
-		(lib_id "power:+3.3V")
+		(lib_id "power:+3V3")
 		(at 252.73 124.46 0)
 		(unit 1)
@@
 			)
 		)
-		(property "Value" "+3.3V"
+		(property "Value" "+3V3"
 			(at 252.73 119.38 0)
 			(show_name no)
@@
 			)
 		)
-		(property "Description" "Power symbol creates a global label with name \"+3.3V\""
+		(property "Description" "Power symbol creates a global label with name \"+3V3\""
 			(at 252.73 124.46 0)
 			(hide yes)
@@
 	)
 	(symbol
-		(lib_id "power:+3.3VA")
+		(lib_id "power:+3V3A")
 		(at 154.94 22.86 0)
 		(unit 1)
@@
 			)
 		)
-		(property "Value" "+3.3VA"
+		(property "Value" "+3V3A"
 			(at 154.94 17.78 0)
 			(show_name no)
@@
 			)
 		)
-		(property "Description" "Power symbol creates a global label with name \"+3.3VA\""
+		(property "Description" "Power symbol creates a global label with name \"+3V3A\""
 			(at 154.94 22.86 0)
 			(hide yes)
@@
 	)
 	(symbol
-		(lib_id "power:+3.3V")
+		(lib_id "power:+3V3")
 		(at 35.56 57.15 0)
 		(unit 1)
@@
 			)
 		)
-		(property "Value" "+3.3V"
+		(property "Value" "+3V3"
 			(at 35.56 52.07 0)
 			(show_name no)
@@
 			)
 		)
-		(property "Description" "Power symbol creates a global label with name \"+3.3V\""
+		(property "Description" "Power symbol creates a global label with name \"+3V3\""
 			(at 35.56 57.15 0)
 			(hide yes)
@@
 	)
 	(symbol
-		(lib_id "power:+3.3VA")
+		(lib_id "power:+3V3A")
 		(at 218.44 124.46 0)
 		(unit 1)
@@
 			)
 		)
-		(property "Value" "+3.3VA"
+		(property "Value" "+3V3A"
 			(at 218.44 119.38 0)
 			(show_name no)
@@
 			)
 		)
-		(property "Description" "Power symbol creates a global label with name \"+3.3VA\""
+		(property "Description" "Power symbol creates a global label with name \"+3V3A\""
 			(at 218.44 124.46 0)
 			(hide yes)
@@
 	)
 	(symbol
-		(lib_id "power:+3.3VA")
+		(lib_id "power:+3V3A")
 		(at 182.88 124.46 0)
 		(unit 1)
@@
 			)
 		)
-		(property "Value" "+3.3VA"
+		(property "Value" "+3V3A"
 			(at 182.88 119.38 0)
 			(show_name no)
@@
 			)
 		)
-		(property "Description" "Power symbol creates a global label with name \"+3.3VA\""
+		(property "Description" "Power symbol creates a global label with name \"+3V3A\""
 			(at 182.88 124.46 0)
 			(hide yes)
@@
 	)
 	(symbol
-		(lib_id "power:+3.3V")
+		(lib_id "power:+3V3")
 		(at 63.5 57.15 0)
 		(unit 1)
@@
 			)
 		)
-		(property "Value" "+3.3V"
+		(property "Value" "+3V3"
 			(at 63.5 52.07 0)
 			(show_name no)
@@
 			)
 		)
-		(property "Description" "Power symbol creates a global label with name \"+3.3V\""
+		(property "Description" "Power symbol creates a global label with name \"+3V3\""
 			(at 63.5 57.15 0)
 			(hide yes)
@@
 	)
 	(symbol
-		(lib_id "power:+3.3VA")
+		(lib_id "power:+3V3A")
 		(at 110.49 40.64 0)
 		(unit 1)
@@
 			)
 		)
-		(property "Value" "+3.3VA"
+		(property "Value" "+3V3A"
 			(at 110.49 35.56 0)
 			(show_name no)
@@
 			)
 		)
-		(property "Description" "Power symbol creates a global label with name \"+3.3VA\""
+		(property "Description" "Power symbol creates a global label with name \"+3V3A\""
 			(at 110.49 40.64 0)
 			(hide yes)
@@
 	)
 	(symbol
-		(lib_id "power:+3.3VA")
+		(lib_id "power:+3V3A")
 		(at 207.01 124.46 0)
 		(unit 1)
@@
 			)
 		)
-		(property "Value" "+3.3VA"
+		(property "Value" "+3V3A"
 			(at 207.01 119.38 0)
 			(show_name no)
@@
 			)
 		)
-		(property "Description" "Power symbol creates a global label with name \"+3.3VA\""
+		(property "Description" "Power symbol creates a global label with name \"+3V3A\""
 			(at 207.01 124.46 0)
 			(hide yes)
@@
 	)
 	(symbol
-		(lib_id "power:+3.3VA")
+		(lib_id "power:+3V3A")
 		(at 264.16 124.46 0)
 		(unit 1)
@@
 			)
 		)
-		(property "Value" "+3.3V"
+		(property "Value" "+3V3"
 			(at 264.16 119.38 0)
 			(show_name no)
@@
 			)
 		)
-		(property "Description" "Power symbol creates a global label with name \"+3.3VA\""
+		(property "Description" "Power symbol creates a global label with name \"+3V3A\""
 			(at 264.16 124.46 0)
 			(hide yes)
@@
 	)
 	(symbol
-		(lib_id "power:+3.3V")
+		(lib_id "power:+3V3")
 		(at 44.45 57.15 0)
 		(unit 1)
@@
 			)
 		)
-		(property "Value" "+3.3V"
+		(property "Value" "+3V3"
 			(at 44.45 52.07 0)
 			(show_name no)
@@
 			)
 		)
-		(property "Description" "Power symbol creates a global label with name \"+3.3V\""
+		(property "Description" "Power symbol creates a global label with name \"+3V3\""
 			(at 44.45 57.15 0)
 			(hide yes)
@@
 	)
 	(symbol
-		(lib_id "power:+3.3V")
+		(lib_id "power:+3V3")
 		(at 53.34 57.15 0)
 		(unit 1)
@@
 			)
 		)
-		(property "Value" "+3.3V"
+		(property "Value" "+3V3"
 			(at 53.34 52.07 0)
 			(show_name no)
@@
 			)
 		)
-		(property "Description" "Power symbol creates a global label with name \"+3.3V\""
+		(property "Description" "Power symbol creates a global label with name \"+3V3\""
 			(at 53.34 57.15 0)
 			(hide yes)
@@
 	)
 	(symbol
-		(lib_id "power:+3.3VA")
+		(lib_id "power:+3V3A")
 		(at 194.31 124.46 0)
 		(unit 1)
@@
 			)
 		)
-		(property "Value" "+3.3VA"
+		(property "Value" "+3V3A"
 			(at 194.31 119.38 0)
 			(show_name no)
@@
 			)
 		)
-		(property "Description" "Power symbol creates a global label with name \"+3.3VA\""
+		(property "Description" "Power symbol creates a global label with name \"+3V3A\""
 			(at 194.31 124.46 0)
 			(hide yes)
