File: Furnace_Controller_V2/sheets/io_expander.kicad_sch (KiCad schematic)
At the start: 2 parts, among them U6 TCA9534

Commit message: Normalize 3.3V net names
Connections:
- net +3.3V renamed +3V3
Changed lines of the file:
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@@
 			)
 		)
-		(property "Value" "+3.3V"
+		(property "Value" "+3V3"
 			(at 157.48 77.47 0)
 			(show_name no)
@@
 			)
 		)
-		(property "Value" "+3.3V"
+		(property "Value" "+3V3"
 			(at 134.62 82.55 0)
 			(show_name no)
