File: Furnace_Controller_V2/sheets/power3v3a.kicad_sch (KiCad schematic)
At the start: 5 parts, among them U7 TPS7A20xxxDBV

Commit message: Normalize 3.3V net names
Connections:
- net +3.3V renamed +3V3
Changed lines of the file:
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@@
 			)
 		)
-		(property "Value" "+3.3V"
+		(property "Value" "+3V3"
 			(at 139.7 68.58 0)
 			(show_name no)
