File: Furnace_Controller_V2/sheets/rs485-module.kicad_sch (KiCad schematic)
At the start: 5 parts, among them U9 THVD2450DR

Commit message: Normalize 3.3V net names
Connections:
- net +3.3V renamed +3V3
Changed lines of the file:
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@@
 			)
 		)
-		(property "Value" "+3.3V"
+		(property "Value" "+3V3"
 			(at 135.89 80.01 0)
 			(show_name no)
@@
 			)
 		)
-		(property "Value" "+3.3V"
+		(property "Value" "+3V3"
 			(at 96.52 59.69 0)
 			(show_name no)
