File: Furnace_Controller_V2/sheets/supervisor_module.kicad_sch (KiCad schematic)
At the start: 6 parts, among them U11 TPS36BA38ACADDFRQ1

Commit message: Normalize 3.3V net names
Connections:
- net +3.3V renamed +3V3
Changed lines of the file:
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@@
 			)
 		)
-		(property "Value" "+3.3V"
+		(property "Value" "+3V3"
 			(at 137.16 109.22 0)
 			(show_name no)
@@
 			)
 		)
-		(property "Value" "+3.3V"
+		(property "Value" "+3V3"
 			(at 133.35 78.74 0)
 			(show_name no)
