File: Furnace_Motherboard_R1/Furnace_Motherboard_R1.kicad_sch (KiCad schematic)
At the start: 0 parts

Commit message: Back up motherboard R1 design and fabrication outputs
Parts:
- added H1, H2, H3, H4: MountingHole, MountingHole:MountingHole_3.2mm_M3, symbol Mechanical:MountingHole
- added J14: Conn_02x12_Odd_Even, Connector_PinSocket_2.54mm:PinSocket_2x12_P2.54mm_Vertical, symbol Connector_Generic:Conn_02x12_Odd_Even
- added R43: 10k, Resistor_SMD:R_0603_1608Metric, symbol Device:R
Connections:
- new net +5V: J14.1 (Pin_1), J14.2 (Pin_2)
- new net CAN_STB: J14.19 (Pin_19)
- new net ETH_CRS_DV: J14.5 (Pin_5)
- new net ETH_MDC: J14.13 (Pin_13)
- new net ETH_MDIO: J14.14 (Pin_14)
- new net ETH_MODULE_PRESENT: J14.17 (Pin_17), R43.1
- new net ETH_PHY_INT_N: J14.16 (Pin_16)
- new net ETH_PHY_RST_N: J14.15 (Pin_15)
- new net ETH_REF_CLK: J14.4 (Pin_4)
- new net ETH_RXD0: J14.6 (Pin_6)
- new net ETH_RXD1: J14.7 (Pin_7)
- new net ETH_TXD0: J14.9 (Pin_9)
- new net ETH_TXD1: J14.10 (Pin_10)
- new net ETH_TX_EN: J14.11 (Pin_11)
- new net EXT_RS485_DE: J14.21 (Pin_21)
- new net EXT_RS485_RX: J14.24 (Pin_24)
- new net EXT_RS485_TX: J14.23 (Pin_23)
- new net FDCAN1_RX: J14.22 (Pin_22)
- new net FDCAN1_TX: J14.20 (Pin_20)
- new net GND: J14.12 (Pin_12), J14.18 (Pin_18), J14.3 (Pin_3), J14.8 (Pin_8), R43.2
Other:
- removed sheet 3V3_LDO
- removed sheet 5v_power_converter
- removed sheet MAIN_MCU_64_PIN
- removed sheet Relay Driver2
- removed sheet Relay Driver3
- removed sheet Relay Driver4
- removed sheet Relay Driver5
- removed sheet Relay Driver6
- removed sheet Relay Driver7
- removed sheet Relay Driver8
- added sheet 24V_TO_5V_BUCK (Power_module.kicad_sch)
- added sheet Relay Driver12 (Relay Driver.kicad_sch)
- added sheet Relay Driver13 (Relay Driver.kicad_sch)
- added sheet Relay Driver14 (Relay Driver.kicad_sch)
- added sheet aux-rs485-module (rs485-module.kicad_sch)
- added sheet power3v3a (power3v3a.kicad_sch)
- sheet Heater Contactor Driver ports: added none; removed RELAY_COIL_IN, RELAY_COIL_SW
- sheet Heater SSR Driver ports: added none; removed RELAY_COIL_IN, RELAY_COIL_SW
- sheet MAIN_MCU ports: added AUX_DO0_CMD, AUX_DO1_CMD, AUX_DO2_CMD, AUX_DO3_CMD, AUX_DO4_CMD, AUX_DO5_CMD, AUX_RS485_DE, AUX_RS485_RX, AUX_RS485_TX, CAN_STB, ETH_CRS_DV, ETH_MDC, ETH_MDIO, ETH_MODULE_PRESENT, ETH_PHY_INT_N, ETH_PHY_RST_N, ETH_REF_CLK, ETH_RXD0, ETH_RXD1, ETH_TXD0, ETH_TXD1, ETH_TX_EN, EXT_RS485_DE, EXT_RS485_RX, EXT_RS485_TX, FDCAN1_RX, FDCAN1_TX, HEATER_CONTACTOR_CMD, HEATER_SSR_CMD, INT_RS485_DE, INT_RS485_RX, INT_RS485_TX, OCTOSPI1_CLK, OCTOSPI1_IO0, OCTOSPI1_IO1, OCTOSPI1_IO2, OCTOSPI1_IO3, OCTOSPI1_NCS, RS422_RX, RS422_TX, SUP_RESET_N, SUP_WDI, VDD, VSS; removed none
- sheet Relay Driver10 ports: added none; removed RELAY_COIL_IN, RELAY_COIL_SW
- sheet Relay Driver11 ports: added none; removed RELAY_COIL_IN, RELAY_COIL_SW
- sheet Relay Driver9 ports: added none; removed RELAY_COIL_IN, RELAY_COIL_SW
- sheet rs-422-module ports: added none; removed A, B, Y, Z
- sheet rs485-module ports: added none; removed A, B
