File: Furnace_Motherboard_R1/Relay Driver.kicad_sch (KiCad schematic)
At the start: 4 parts, among them Q1 20N04-MS

Commit message: Back up motherboard R1 design and fabrication outputs
Parts:
- removed D3: SM4007, Diode_SMD:D_SOD-123, symbol Diode:SM4007
- added D1: US1B, Diode_SMD:D_SMA, symbol Diode:US1B
- added D15: LED, LED_SMD:LED_0603_1608Metric, symbol Device:LED
- added J1: Conn_01x02, Connector_Phoenix_MC:PhoenixContact_MC_1,5_2-G-3.5_1x02_P3.50mm_Horizontal, symbol Connector_Generic:Conn_01x02
- added R44: 150, Resistor_SMD:R_0603_1608Metric, symbol Device:R
- Q1: value 20N04-MS -> BSS606N
- renumbered R10 to R1, R11 to R2
Connections:
- net RELAY_CTRL: now also D15.2 (A)
- net VSS: now also R44.1
- net RELAY_COIL_SW: no longer names the net of Q1.2 (D)
- net RELAY_COIL_SW: now also D1.2 (A), J1.1 (Pin_1)
- new net: D1.1 (K), J1.2 (Pin_2)
- new net: D15.1 (K), R44.2
