File: Furnace_Motherboard_R1/ex_flash_module.kicad_sch (KiCad schematic)
At the start: 6 parts, among them U6 W25Q128JVS

Commit message: Back up motherboard R1 design and fabrication outputs
Parts:
- R30: renamed from R36; footprint Resistor_SMD:R_0201_0603Metric -> Resistor_SMD:R_0603_1608Metric
- R31: renamed from R35; footprint Resistor_SMD:R_0201_0603Metric -> Resistor_SMD:R_0603_1608Metric
- R32: renamed from R34; footprint Resistor_SMD:R_0201_0603Metric -> Resistor_SMD:R_0603_1608Metric
- renumbered C22 to C24, C21 to C25, U6 to U5
Changed lines of the file:
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@@
 		(dnp no)
 		(fields_autoplaced yes)
-		(property "Reference" "C22"
+		(property "Reference" "C24"
 			(at 83.82 66.0399 0)
 			(show_name no)
@@
 			(project "Furnace_Motherboard_R1"
 				(path "/43d4b116-7476-4705-a5a8-f2a03f21058e/3172dcfb-3c78-437a-858c-6ce7db97375b"
-					(reference "C22")
+					(reference "C24")
 					(unit 1)
 				)
@@
 		(dnp no)
 		(fields_autoplaced yes)
-		(property "Reference" "R35"
+		(property "Reference" "R31"
 			(at 124.46 62.2299 0)
 			(show_name no)
@@
 			)
 		)
-		(property "Footprint" "Resistor_SMD:R_0201_0603Metric"
+		(property "Footprint" "Resistor_SMD:R_0603_1608Metric"
 			(at 120.142 63.5 90)
 			(hide yes)
@@
 			(project "Furnace_Motherboard_R1"
 				(path "/43d4b116-7476-4705-a5a8-f2a03f21058e/3172dcfb-3c78-437a-858c-6ce7db97375b"
-					(reference "R35")
+					(reference "R31")
 					(unit 1)
 				)
@@
 		(dnp no)
 		(fields_autoplaced yes)
-		(property "Reference" "C21"
+		(property "Reference" "C25"
 			(at 93.98 66.0399 0)
 			(show_name no)
@@
 			(project "Furnace_Motherboard_R1"
 				(path "/43d4b116-7476-4705-a5a8-f2a03f21058e/3172dcfb-3c78-437a-858c-6ce7db97375b"
-					(reference "C21")
+					(reference "C25")
 					(unit 1)
 				)
@@
 		(dnp no)
 		(fields_autoplaced yes)
-		(property "Reference" "R34"
+		(property "Reference" "R32"
 			(at 133.35 62.2299 0)
 			(show_name no)
@@
 			)
 		)
-		(property "Footprint" "Resistor_SMD:R_0201_0603Metric"
+		(property "Footprint" "Resistor_SMD:R_0603_1608Metric"
 			(at 129.032 63.5 90)
 			(hide yes)
@@
 			(project "Furnace_Motherboard_R1"
 				(path "/43d4b116-7476-4705-a5a8-f2a03f21058e/3172dcfb-3c78-437a-858c-6ce7db97375b"
-					(reference "R34")
+					(reference "R32")
 					(unit 1)
 				)
@@
 		(dnp no)
 		(fields_autoplaced yes)
-		(property "Reference" "R36"
+		(property "Reference" "R30"
 			(at 115.57 62.2299 0)
 			(show_name no)
@@
 			)
 		)
-		(property "Footprint" "Resistor_SMD:R_0201_0603Metric"
+		(property "Footprint" "Resistor_SMD:R_0603_1608Metric"
 			(at 111.252 63.5 90)
 			(hide yes)
@@
 			(project "Furnace_Motherboard_R1"
 				(path "/43d4b116-7476-4705-a5a8-f2a03f21058e/3172dcfb-3c78-437a-858c-6ce7db97375b"
-					(reference "R36")
+					(reference "R30")
 					(unit 1)
 				)
@@
 		(dnp no)
 		(fields_autoplaced yes)
-		(property "Reference" "U6"
+		(property "Reference" "U5"
 			(at 157.48 77.4699 0)
 			(show_name no)
@@
 			(project "Furnace_Motherboard_R1"
 				(path "/43d4b116-7476-4705-a5a8-f2a03f21058e/3172dcfb-3c78-437a-858c-6ce7db97375b"
-					(reference "U6")
-					(unit 1)
-				)
+					(reference "U5")
+					(unit 1)
+				)
