File: Furnace_Motherboard_R1/main_mcu.kicad_sch (KiCad schematic)
At the start: 20 parts, among them J2 Conn_02x07_Odd_Even, U1 STM32H563VITx

Commit message: Back up motherboard R1 design and fabrication outputs
Parts:
- removed TP1, TP2: TestPoint, TestPoint:TestPoint_Pad_D1.0mm, symbol Connector:TestPoint
- added C1: 100n, Capacitor_SMD:C_0603_1608Metric, symbol Device:C
- added C10, C12: C, Capacitor_SMD:C_0603_1608Metric, symbol Device:C
- added Y1: Crystal_GND24_Small, Crystal:Crystal_SMD_3225-4Pin_3.2x2.5mm, symbol Device:Crystal_GND24_Small
- renumbered C13 to C11, C1 to C13, C2 to C14, C14 to C2, C12 to C3, C11 to C4, C7 to C5, C8 to C6, C15 to C7, C9 to C8, C10 to C9, J2 to J3, R3 to R5, R2 to R6, R1 to R7
Connections:
- net VDD: now also R7.1, U1.100 (VDD), U1.11 (VDD), U1.28 (VDD), U1.6 (VBAT), U1.73 (VDDUSB), U1.75 (VDD); no longer C3.1
- net VDDA: now also C3.1, C1.1
- net VSS: now also C1.2, C10.2, C12.2, Y1.2 (G), Y1.4 (G)
- net RCC_OSC_IN: now reaches U1.12 (PH0)
- net RCC_OSC_IN: now also C12.1, Y1.3
- net RCC_OSC_OUT: now reaches U1.13 (PH1)
- net RCC_OSC_OUT: now also C10.1, Y1.1
- net RS422_RX: now reaches U1.81 (PD0)
- net RS422_TX: now reaches U1.82 (PD1)
- net AUX_DO6_CMD: no longer names the net of U1.43 (PE12)
- net AUX_DO7_CMD: no longer names the net of U1.44 (PE13)
- net AUX_DO8_CMD: no longer names the net of U1.45 (PE14)
- net AUX_DO9_CMD: no longer names the net of U1.46 (PE15)
- net SUP_WID renamed SUP_WDI
- net UART5_DE renamed AUX_RS485_DE
- net UART5_RX renamed AUX_RS485_RX
- net UART5_TX renamed AUX_RS485_TX
- net USART1_RX: no longer names the net of U1.69 (PA10)
- net USART1_TX: no longer names the net of U1.68 (PA9)
- net USART2_DE renamed INT_RS485_DE
- net USART2_RX renamed INT_RS485_RX
- net USART2_TX renamed INT_RS485_TX
- net USART3_DE renamed EXT_RS485_DE
- net USART3_RX renamed EXT_RS485_RX
- net USART3_TX renamed EXT_RS485_TX
- no-connect marks 3 -> 33
Other:
- moved on the sheet: C13, C14
