File: Furnace_Motherboard_R1/rs-422-module.kicad_sch (KiCad schematic)
At the start: 9 parts, among them U4 PTHVD2452VDR

Commit message: Back up motherboard R1 design and fabrication outputs
Parts:
- added D3, D4: SM712_SOT23, Package_TO_SOT_SMD:SOT-23, symbol Diode:SM712_SOT23
- added J4: Conn_01x05, Connector_Phoenix_MC:PhoenixContact_MC_1,5_5-G-3.5_1x05_P3.50mm_Horizontal, symbol Connector_Generic:Conn_01x05
- added R12: 120, Resistor_SMD:R_0603_1608Metric, symbol Device:R
- added R13, R14: 15, Resistor_SMD:R_0603_1608Metric, symbol Device:R
- C17: renamed from C18; value 10u -> 1u
- C18: renamed from C19; value 10u -> 1u
- renumbered C16 to C15, C17 to C16, R6 to R10, R7 to R11, R4 to R8, R5 to R9, U4 to U2
Connections:
- net A: now also D3.1 (A1), J4.5 (Pin_5), R12.1
- net B: now also D3.2 (A2), J4.4 (Pin_4), R12.2
- net GND: now also D3.3 (common), D4.3 (common), J4.1 (Pin_1)
- net Y: now also D4.2 (A2), J4.2 (Pin_2), R13.1; no longer U2.9 (Y)
- net Z: now also D4.1 (A1), J4.3 (Pin_3), R14.1; no longer U2.10 (Z)
- new net: R14.2, U2.10 (Z)
- new net: R13.2, U2.9 (Y)
Other:
- moved on the sheet: C15, C16, C17, C18, R10, R11, R8, R9
