File: Furnace_Motherboard_R1/rs485-module.kicad_sch (KiCad schematic)
At the start: 5 parts, among them U5 THVD2450DR

Commit message: Back up motherboard R1 design and fabrication outputs
Parts:
- added J5: Conn_01x03, Connector_Phoenix_MC:PhoenixContact_MC_1,5_3-G-3.5_1x03_P3.50mm_Horizontal, symbol Connector_Generic:Conn_01x03
- added R17: 120, Resistor_SMD:R_0603_1608Metric, symbol Device:R
- renumbered C20 to C19, D2 to D5, R8 to R15, R9 to R16, U5 to U3
Connections:
- net GND: now also J5.1 (Pin_1)
- net A: no longer names the net of D5.2 (A2), R16.2
- net A: now also J5.2 (Pin_2), R17.2
- net B: no longer names the net of D5.1 (A1), R15.2
- net B: now also J5.3 (Pin_3), R17.1
