File: Furnace_Motherboard_R1/supervisor_module.kicad_sch (KiCad schematic)
At the start: 6 parts, among them U7 TPS36BA38ACADDFRQ1

Commit message: Back up motherboard R1 design and fabrication outputs
Parts:
- renumbered C23 to C26, C24 to C27, C25 to C28, R37 to R33, R38 to R34, U7 to U6
Changed lines of the file:
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@@
 		(dnp no)
 		(fields_autoplaced yes)
-		(property "Reference" "R38"
+		(property "Reference" "R34"
 			(at 127 86.3599 0)
 			(show_name no)
@@
 			(project "Furnace_Motherboard_R1"
 				(path "/43d4b116-7476-4705-a5a8-f2a03f21058e/57b4129e-afdd-4a4f-bda5-255cd6f5afd3"
-					(reference "R38")
+					(reference "R34")
 					(unit 1)
 				)
@@
 		(in_pos_files yes)
 		(dnp no)
-		(property "Reference" "C25"
+		(property "Reference" "C28"
 			(at 125.73 48.2599 0)
 			(show_name no)
@@
 			(project "Furnace_Motherboard_R1"
 				(path "/43d4b116-7476-4705-a5a8-f2a03f21058e/57b4129e-afdd-4a4f-bda5-255cd6f5afd3"
-					(reference "C25")
+					(reference "C28")
 					(unit 1)
 				)
@@
 		(dnp no)
 		(fields_autoplaced yes)
-		(property "Reference" "U7"
+		(property "Reference" "U6"
 			(at 166.37 58.42 0)
 			(show_name no)
@@
 			(project "Furnace_Motherboard_R1"
 				(path "/43d4b116-7476-4705-a5a8-f2a03f21058e/57b4129e-afdd-4a4f-bda5-255cd6f5afd3"
-					(reference "U7")
+					(reference "U6")
 					(unit 1)
 				)
@@
 		(in_pos_files yes)
 		(dnp no)
-		(property "Reference" "C24"
+		(property "Reference" "C27"
 			(at 107.95 86.3599 0)
 			(show_name no)
@@
 			(project "Furnace_Motherboard_R1"
 				(path "/43d4b116-7476-4705-a5a8-f2a03f21058e/57b4129e-afdd-4a4f-bda5-255cd6f5afd3"
-					(reference "C24")
+					(reference "C27")
 					(unit 1)
 				)
@@
 		(dnp no)
 		(fields_autoplaced yes)
-		(property "Reference" "R37"
+		(property "Reference" "R33"
 			(at 119.38 86.3599 0)
 			(show_name no)
@@
 			(project "Furnace_Motherboard_R1"
 				(path "/43d4b116-7476-4705-a5a8-f2a03f21058e/57b4129e-afdd-4a4f-bda5-255cd6f5afd3"
-					(reference "R37")
+					(reference "R33")
 					(unit 1)
 				)
@@
 		(in_pos_files yes)
 		(dnp no)
-		(property "Reference" "C23"
+		(property "Reference" "C26"
 			(at 95.25 86.3599 0)
 			(show_name no)
@@
 			(project "Furnace_Motherboard_R1"
 				(path "/43d4b116-7476-4705-a5a8-f2a03f21058e/57b4129e-afdd-4a4f-bda5-255cd6f5afd3"
-					(reference "C23")
-					(unit 1)
-				)
+					(reference "C26")
+					(unit 1)
+				)
